Commit message: Upload current wall climber update

File: src/wall_climber/urdf/simple_pen_mount.xacro (robot description, xacro)
@@ -5,90 +5,85 @@
         <xacro:property name="carriage_cfg" value="${robot_cfg['carriage']}"/>
         <xacro:property name="pen_cfg" value="${robot_cfg['pen']}"/>
-        <!-- After the launch rotation, URDF -Z faces the board and URDF +X points right. -->
+        <!-- After launch rotation, URDF -Z faces the board and URDF +X points right. -->
         <xacro:property name="pen_local_y" value="${-carriage_cfg['pen_offset_y']}"/>
-        <!-- Keep the shoulder root inside the orange chassis and let only the linkage protrude. -->
-        <xacro:property name="arm_mount_x" value="${(carriage_cfg['width'] / 2.0) - 0.014}"/>
-        <xacro:property name="arm_mount_z" value="${-(carriage_cfg['depth'] / 2.0) + 0.008}"/>
-        <xacro:property name="slide_origin_z" value="-0.006"/>
-        <!-- ════════════════  SHOULDER (arm_mount)  ════════════════ -->
-        <xacro:property name="shoulder_size_x" value="0.020"/>
-        <xacro:property name="shoulder_size_y" value="0.040"/>
-        <xacro:property name="shoulder_size_z" value="0.010"/>
-        <xacro:property name="shoulder_flange_x" value="0.028"/>
-        <xacro:property name="shoulder_flange_y" value="0.046"/>
-        <xacro:property name="shoulder_flange_z" value="0.0028"/>
-        <xacro:property name="shoulder_bridge_x" value="0.020"/>
-        <xacro:property name="shoulder_bridge_y" value="0.014"/>
-        <xacro:property name="shoulder_bridge_z" value="0.005"/>
-        <xacro:property name="bolt_radius" value="0.002"/>
-        <xacro:property name="bolt_length" value="0.003"/>
-        <!-- ════════════════  LIFT STAGE  ════════════════ -->
+        <xacro:property name="arm_mount_x" value="${(carriage_cfg['width'] / 2.0) - 0.018}"/>
+        <xacro:property name="arm_mount_z" value="${-(carriage_cfg['depth'] / 2.0) + 0.0075}"/>
+        <xacro:property name="slide_origin_z" value="-0.0082"/>
+        <!-- Shoulder plate -->
+        <xacro:property name="shoulder_size_x" value="0.021"/>
+        <xacro:property name="shoulder_size_y" value="0.054"/>
+        <xacro:property name="shoulder_size_z" value="0.0074"/>
+        <xacro:property name="shoulder_flange_x" value="0.027"/>
+        <xacro:property name="shoulder_flange_y" value="0.060"/>
+        <xacro:property name="shoulder_flange_z" value="0.0024"/>
+        <xacro:property name="shoulder_bridge_x" value="0.014"/>
+        <xacro:property name="shoulder_bridge_y" value="0.018"/>
+        <xacro:property name="shoulder_bridge_z" value="0.0046"/>
+        <!-- Lift carriage -->
         <xacro:property name="lift_block_x" value="0.018"/>
-        <xacro:property name="lift_block_y" value="0.026"/>
-        <xacro:property name="lift_block_z" value="0.008"/>
-        <xacro:property name="lift_shroud_x" value="0.036"/>
-        <xacro:property name="lift_shroud_y" value="0.020"/>
-        <xacro:property name="lift_shroud_z" value="0.004"/>
+        <xacro:property name="lift_block_y" value="0.046"/>
+        <xacro:property name="lift_block_z" value="0.0062"/>
+        <xacro:property name="lift_cover_x" value="0.032"/>
+        <xacro:property name="lift_cover_y" value="0.031"/>
+        <xacro:property name="lift_cover_z" value="0.0034"/>
         <xacro:property name="rail_radius" value="${pen_cfg['support_radius'] * 0.42}"/>
         <xacro:property name="rail_length" value="0.020"/>
-        <xacro:property name="rail_offset_y" value="0.0048"/>
-        <!-- ════════════════  FOREARM (shortened)  ════════════════ -->
-        <xacro:property name="forearm_joint_x" value="0.020"/>
+        <xacro:property name="rail_offset_y" value="0.0058"/>
+        <!-- Forearm / wrist plate -->
+        <xacro:property name="forearm_joint_x" value="0.028"/>
         <xacro:property name="forearm_size_x" value="0.044"/>
-        <xacro:property name="forearm_size_y" value="0.018"/>
-        <xacro:property name="forearm_size_z" value="0.004"/>
-        <xacro:property name="forearm_rib_y" value="0.0032"/>
-        <xacro:property name="forearm_rib_z" value="0.0018"/>
-        <!-- ════════════════  WRIST (shortened)  ════════════════ -->
+        <xacro:property name="forearm_size_y" value="0.034"/>
+        <xacro:property name="forearm_size_z" value="0.0032"/>
+        <xacro:property name="forearm_plate_gap" value="0.011"/>
+        <xacro:property name="forearm_plate_y" value="0.0068"/>
+        <xacro:property name="forearm_plate_z" value="0.0032"/>
+        <xacro:property name="forearm_bridge_x" value="0.010"/>
+        <xacro:property name="forearm_bridge_y" value="0.022"/>
+        <xacro:property name="forearm_bridge_z" value="0.0036"/>
         <xacro:property name="wrist_joint_x" value="0.024"/>
         <xacro:property name="wrist_size_x" value="0.014"/>
-        <xacro:property name="wrist_size_y" value="0.028"/>
-        <xacro:property name="wrist_size_z" value="0.006"/>
-        <!-- ════════════════  GRIPPER (split-ring clamp)  ════════════════ -->
-        <xacro:property name="pen_holder_x" value="0.028"/>
-        <xacro:property name="pen_holder_z" value="0.000"/>
-        <xacro:property name="clamp_base_x" value="0.012"/>
-        <xacro:property name="clamp_base_y" value="0.012"/>
-        <xacro:property name="clamp_base_z" value="0.004"/>
-        <xacro:property name="clamp_link_x" value="0.020"/>
-        <xacro:property name="clamp_link_y" value="0.0028"/>
-        <xacro:property name="clamp_link_z" value="0.0032"/>
-        <xacro:property name="clamp_ring_radius" value="${pen_cfg['radius'] + 0.0042}"/>
-        <xacro:property name="clamp_ring_length" value="0.0046"/>
-        <xacro:property name="clamp_ring_x" value="${pen_holder_x - 0.004}"/>
-        <xacro:property name="clamp_ring_z" value="0.013"/>
-        <xacro:property name="clamp_cap_radius" value="0.0024"/>
-        <xacro:property name="jaw_body_size_x" value="0.012"/>
-        <xacro:property name="jaw_body_size_y" value="0.0040"/>
-        <xacro:property name="jaw_body_size_z" value="0.014"/>
-        <xacro:property name="jaw_closed_offset_y" value="${pen_cfg['radius'] + 0.0024}"/>
-        <xacro:property name="jaw_open_travel" value="${pen_cfg['gripper_open_position']}"/>
-        <xacro:property name="jaw_velocity" value="${pen_cfg['gripper_velocity']}"/>
-        <!-- Gripper origin offsets (applied via fixed joints to avoid Webots Pose bug) -->
-        <xacro:property name="grip_origin_x" value="0.003"/>
-        <xacro:property name="grip_origin_z" value="0.000"/>
-        <!-- ════════════════  MARKER PEN (clean, like pantograph)  ════════════════ -->
+        <xacro:property name="wrist_size_y" value="0.032"/>
+        <xacro:property name="wrist_size_z" value="0.0054"/>
+        <xacro:property name="wrist_plate_x" value="0.020"/>
+        <xacro:property name="wrist_plate_y" value="0.028"/>
+        <xacro:property name="wrist_plate_z" value="0.0032"/>
+        <!-- Pen holder / C-cradle -->
+        <xacro:property name="pen_holder_x" value="0.024"/>
+        <xacro:property name="pen_holder_z" value="0.0"/>
+        <xacro:property name="holder_stem_x" value="0.020"/>
+        <xacro:property name="holder_stem_y" value="0.012"/>
+        <xacro:property name="holder_stem_z" value="0.007"/>
+        <xacro:property name="cradle_center_z" value="0.0120"/>
+        <xacro:property name="cradle_back_x" value="-0.0070"/>
+        <xacro:property name="cradle_back_size_x" value="0.0048"/>
+        <xacro:property name="cradle_back_size_y" value="0.0200"/>
+        <xacro:property name="cradle_back_size_z" value="0.0130"/>
+        <xacro:property name="cradle_arm_size_x" value="0.0130"/>
+        <xacro:property name="cradle_arm_size_y" value="0.0034"/>
+        <xacro:property name="cradle_arm_size_z" value="0.0130"/>
+        <xacro:property name="cradle_arm_center_x" value="0.0010"/>
+        <xacro:property name="cradle_arm_offset_y" value="${pen_cfg['radius'] + 0.0012}"/>
+        <xacro:property name="cradle_web_x" value="0.007"/>
+        <xacro:property name="cradle_web_y" value="0.010"/>
+        <xacro:property name="cradle_web_z" value="0.010"/>
+        <!-- Marker pen -->
         <xacro:property name="marker_r" value="${pen_cfg['radius']}"/>
         <xacro:property name="marker_h" value="${pen_cfg['mount_length']}"/>
-        <xacro:property name="marker_body_front_z" value="0.004"/>
+        <xacro:property name="marker_body_front_z" value="-0.0036"/>
         <xacro:property name="marker_body_center_z" value="${marker_body_front_z + (marker_h / 2.0)}"/>
-        <xacro:property name="marker_front_band_length" value="0.006"/>
+        <xacro:property name="marker_front_band_length" value="0.007"/>
         <xacro:property name="marker_front_band_z" value="${marker_body_front_z + (marker_front_band_length / 2.0)}"/>
-        <xacro:property name="marker_back_cap_length" value="0.006"/>
+        <xacro:property name="marker_back_cap_length" value="0.008"/>
         <xacro:property name="marker_back_cap_z" value="${marker_body_front_z + marker_h - (marker_back_cap_length / 2.0)}"/>
-        <!-- ════════════════  PEN TIP (from pantograph — simple)  ════════════════ -->
-        <xacro:property name="marker_tip_r" value="0.0035"/>
-        <xacro:property name="marker_tip_h" value="0.012"/>
+        <!-- Tip -->
+        <xacro:property name="marker_tip_r" value="0.0033"/>
+        <xacro:property name="marker_tip_h" value="0.0028"/>
         <xacro:property name="marker_tip_contact_r" value="${pen_cfg['tip_radius']}"/>
         <xacro:property name="tip_contact_z" value="${pen_cfg['tip_local_z']}"/>
-        <xacro:property name="marker_tip_front_z"
-            value="${tip_contact_z - marker_tip_contact_r}"/>
+        <xacro:property name="marker_tip_front_z" value="${tip_contact_z - marker_tip_contact_r}"/>
         <xacro:property name="marker_tip_cylinder_z"
             value="${marker_tip_front_z + marker_tip_contact_r + (marker_tip_h / 2.0)}"/>
         <xacro:property name="support_center_z"
-            value="${tip_contact_z + marker_tip_contact_r + 0.0040}"/>
-        <!-- ═══════════════════════════════════════════════════════ -->
-        <!--                 SHOULDER JOINT & LINK                  -->
-        <!-- ═══════════════════════════════════════════════════════ -->
+            value="${tip_contact_z + marker_tip_contact_r + 0.0044}"/>
         <joint name="arm_mount_joint" type="fixed">
             <parent link="chassis"/>
@@ -98,10 +93,9 @@
         <link name="arm_mount">
             <visual>
-                <origin xyz="0 0 0" rpy="0 0 0"/>
                 <geometry>
                     <box size="${shoulder_size_x} ${shoulder_size_y} ${shoulder_size_z}"/>
                 </geometry>
                 <material name="arm_mount_housing">
-                    <color rgba="0.14 0.16 0.20 1.0"/>
+                    <color rgba="0.17 0.19 0.23 1.0"/>
                 </material>
             </visual>
@@ -112,63 +106,27 @@
                 </geometry>
                 <material name="arm_mount_flange">
-                    <color rgba="0.30 0.33 0.38 1.0"/>
-                </material>
-            </visual>
-            <visual>
-                <origin xyz="${shoulder_bridge_x * 0.50} 0 ${-0.001}" rpy="0 0 0"/>
+                    <color rgba="0.33 0.36 0.41 1.0"/>
+                </material>
+            </visual>
+            <visual>
+                <origin xyz="${shoulder_bridge_x * 0.46} 0 -0.001" rpy="0 0 0"/>
                 <geometry>
                     <box size="${shoulder_bridge_x} ${shoulder_bridge_y} ${shoulder_bridge_z}"/>
                 </geometry>
                 <material name="arm_mount_bridge">
-                    <color rgba="0.20 0.23 0.28 1.0"/>
-                </material>
-            </visual>
-            <visual>
-                <origin xyz="${shoulder_flange_x * 0.38} ${shoulder_flange_y * 0.38} ${(shoulder_size_z / 2.0) + 0.001}" rpy="0 0 0"/>
-                <geometry><cylinder radius="${bolt_radius}" length="${bolt_length}"/></geometry>
-                <material name="bolt_chrome"><color rgba="0.72 0.75 0.80 1.0"/></material>
-            </visual>
-            <visual>
-                <origin xyz="${-shoulder_flange_x * 0.38} ${shoulder_flange_y * 0.38} ${(shoulder_size_z / 2.0) + 0.001}" rpy="0 0 0"/>
-                <geometry><cylinder radius="${bolt_radius}" length="${bolt_length}"/></geometry>
-                <material name="bolt_chrome"><color rgba="0.72 0.75 0.80 1.0"/></material>
-            </visual>
-            <visual>
-                <origin xyz="${shoulder_flange_x * 0.38} ${-shoulder_flange_y * 0.38} ${(shoulder_size_z / 2.0) + 0.001}" rpy="0 0 0"/>
-                <geometry><cylinder radius="${bolt_radius}" length="${bolt_length}"/></geometry>
-                <material name="bolt_chrome"><color rgba="0.72 0.75 0.80 1.0"/></material>
-            </visual>
-            <visual>
-                <origin xyz="${-shoulder_flange_x * 0.38} ${-shoulder_flange_y * 0.38} ${(shoulder_size_z / 2.0) + 0.001}" rpy="0 0 0"/>
-                <geometry><cylinder radius="${bolt_radius}" length="${bolt_length}"/></geometry>
-                <material name="bolt_chrome"><color rgba="0.72 0.75 0.80 1.0"/></material>
-            </visual>
-            <visual>
-                <origin xyz="${shoulder_size_x * 0.10} 0 ${shoulder_size_z * 0.14}" rpy="0 0 0"/>
-                <geometry>
-                    <box size="${shoulder_size_x * 0.42} ${shoulder_size_y * 0.58} ${shoulder_size_z * 0.14}"/>
-                </geometry>
-                <material name="arm_mount_highlight">
-                    <color rgba="0.44 0.48 0.55 1.0"/>
-                </material>
-            </visual>
-            <collision>
-                <origin xyz="${shoulder_bridge_x * 0.18} 0 0" rpy="0 0 0"/>
-                <geometry>
-                    <box size="${shoulder_size_x + (shoulder_bridge_x * 0.35)} ${shoulder_size_y} ${shoulder_size_z}"/>
-                </geometry>
-            </collision>
-            <inertial>
-                <origin xyz="0 0 0" rpy="0 0 0"/>
+                    <color rgba="0.24 0.27 0.32 1.0"/>
+                </material>
+            </visual>
+            <collision>
+                <origin xyz="${shoulder_bridge_x * 0.20} 0 0" rpy="0 0 0"/>
+                <geometry>
+                    <box size="${shoulder_size_x + (shoulder_bridge_x * 0.40)} ${shoulder_size_y} ${shoulder_size_z}"/>
+                </geometry>
+            </collision>
+            <inertial>
                 <mass value="0.05"/>
                 <inertia ixx="4.0e-5" ixy="0.0" ixz="0.0" iyy="4.0e-5" iyz="0.0" izz="4.0e-5"/>
             </inertial>
         </link>
-        <!-- ═══════════════════════════════════════════════════════ -->
-        <!--  PEN SLIDE: fixed offset link → prismatic (origin=0)   -->
-        <!-- ═══════════════════════════════════════════════════════ -->
-        <!-- Fixed joint absorbs the slide_origin_z offset so the
-             prismatic joint has origin (0,0,0) — avoids the Webots
-             R2023b "Skipped unknown Pose field in SliderJoint" bug. -->
         <joint name="pen_slide_origin_joint" type="fixed">
             <parent link="arm_mount"/>
@@ -178,5 +136,4 @@
         <link name="pen_slide_origin">
             <inertial>
-                <origin xyz="0 0 0" rpy="0 0 0"/>
                 <mass value="0.001"/>
                 <inertia ixx="1e-8" ixy="0" ixz="0" iyy="1e-8" iyz="0" izz="1e-8"/>
@@ -193,43 +150,30 @@
         <link name="arm_lift_stage">
             <visual>
-                <origin xyz="0.006 0 0" rpy="0 0 0"/>
+                <origin xyz="0.007 0 0" rpy="0 0 0"/>
                 <geometry>
                     <box size="${lift_block_x} ${lift_block_y} ${lift_block_z}"/>
                 </geometry>
                 <material name="arm_lift_block">
-                    <color rgba="0.18 0.21 0.26 1.0"/>
-                </material>
-            </visual>
-            <visual>
-                <origin xyz="${lift_shroud_x * 0.45} 0 ${-0.001}" rpy="0 0 0"/>
-                <geometry>
-                    <box size="${lift_shroud_x} ${lift_shroud_y} ${lift_shroud_z}"/>
-                </geometry>
-                <material name="arm_lift_shroud">
-                    <color rgba="0.23 0.27 0.32 1.0"/>
-                </material>
-            </visual>
-            <visual>
-                <origin xyz="0.002 ${rail_offset_y} 0" rpy="0 1.5708 0"/>
-                <geometry>
-                    <cylinder radius="${rail_radius}" length="${rail_length}"/>
-                </geometry>
-                <material name="arm_rail_polished">
-                    <color rgba="0.70 0.73 0.78 1.0"/>
-                </material>
-            </visual>
-            <visual>
-                <origin xyz="0.002 ${-rail_offset_y} 0" rpy="0 1.5708 0"/>
-                <geometry>
-                    <cylinder radius="${rail_radius}" length="${rail_length}"/>
-                </geometry>
-                <material name="arm_rail_polished">
-                    <color rgba="0.70 0.73 0.78 1.0"/>
-                </material>
-            </visual>
-            <visual>
-                <origin xyz="${lift_block_x * 0.45} ${lift_block_y * 0.34} ${lift_block_z * 0.26}" rpy="0 0 0"/>
-                <geometry><sphere radius="0.0015"/></geometry>
-                <material name="arm_led_green"><color rgba="0.10 0.90 0.30 1.0"/></material>
+                    <color rgba="0.21 0.24 0.29 1.0"/>
+                </material>
+            </visual>
+            <visual>
+                <origin xyz="${lift_cover_x * 0.42} 0 -0.0008" rpy="0 0 0"/>
+                <geometry>
+                    <box size="${lift_cover_x} ${lift_cover_y} ${lift_cover_z}"/>
+                </geometry>
+                <material name="arm_lift_cover">
+                    <color rgba="0.38 0.43 0.49 1.0"/>
+                </material>
+            </visual>
+            <visual>
+                <origin xyz="0.003 ${rail_offset_y} 0" rpy="0 1.5708 0"/>
+                <geometry><cylinder radius="${rail_radius}" length="${rail_length}"/></geometry>
+                <material name="arm_rail_polished"><color rgba="0.70 0.73 0.78 1.0"/></material>
+            </visual>
+            <visual>
+                <origin xyz="0.003 ${-rail_offset_y} 0" rpy="0 1.5708 0"/>
+                <geometry><cylinder radius="${rail_radius}" length="${rail_length}"/></geometry>
+                <material name="arm_rail_polished"><color rgba="0.70 0.73 0.78 1.0"/></material>
             </visual>
             <collision>
@@ -240,12 +184,8 @@
             </collision>
             <inertial>
-                <origin xyz="0 0 0" rpy="0 0 0"/>
-                <mass value="0.04"/>
-                <inertia ixx="3.0e-5" ixy="0.0" ixz="0.0" iyy="3.0e-5" iyz="0.0" izz="3.0e-5"/>
-            </inertial>
-        </link>
-        <!-- ═══════════════════════════════════════════════════════ -->
-        <!--                       FOREARM                          -->
-        <!-- ═══════════════════════════════════════════════════════ -->
+                <mass value="0.03"/>
+                <inertia ixx="2.0e-5" ixy="0.0" ixz="0.0" iyy="2.0e-5" iyz="0.0" izz="2.0e-5"/>
+            </inertial>
+        </link>
         <joint name="arm_forearm_joint" type="fixed">
             <parent link="arm_lift_stage"/>
@@ -255,41 +195,32 @@
         <link name="arm_forearm">
             <visual>
-                <origin xyz="0 ${forearm_size_y * 0.28} 0" rpy="0 0 0"/>
-                <geometry>
-                    <box size="${forearm_size_x} ${forearm_size_y * 0.34} ${forearm_size_z}"/>
-                </geometry>
-                <material name="arm_forearm_body">
-                    <color rgba="0.50 0.78 0.83 1.0"/>
-                </material>
-            </visual>
-            <visual>
-                <origin xyz="0 ${-forearm_size_y * 0.28} 0" rpy="0 0 0"/>
-                <geometry>
-                    <box size="${forearm_size_x} ${forearm_size_y * 0.34} ${forearm_size_z}"/>
+                <origin xyz="${forearm_size_x * 0.48} ${forearm_plate_gap} 0" rpy="0 0 0"/>
+                <geometry>
+                    <box size="${forearm_size_x} ${forearm_plate_y} ${forearm_plate_z}"/>
+                </geometry>
+                <material name="arm_forearm_plate">
+                    <color rgba="0.49 0.58 0.64 1.0"/>
+                </material>
+            </visual>
+            <visual>
+                <origin xyz="${forearm_size_x * 0.48} ${-forearm_plate_gap} 0" rpy="0 0 0"/>
+                <geometry>
+                    <box size="${forearm_size_x} ${forearm_plate_y} ${forearm_plate_z}"/>
+                </geometry>
+                <material name="arm_forearm_plate">
+                    <color rgba="0.49 0.58 0.64 1.0"/>
+                </material>
+            </visual>
+            <visual>
+                <origin xyz="${forearm_size_x * 0.68} 0 0" rpy="0 0 0"/>
+                <geometry>
+                    <box size="${forearm_bridge_x} ${forearm_bridge_y} ${forearm_bridge_z}"/>
                 </geometry>
                 <material name="arm_forearm_rib">
-                    <color rgba="0.50 0.78 0.83 1.0"/>
-                </material>
-            </visual>
-            <visual>
-                <origin xyz="0 ${forearm_size_y * 0.36} ${forearm_size_z * 0.34}" rpy="0 0 0"/>
-                <geometry>
-                    <box size="${forearm_size_x * 0.82} ${forearm_rib_y} ${forearm_rib_z}"/>
-                </geometry>
-                <material name="arm_forearm_rib">
-                    <color rgba="0.34 0.38 0.45 1.0"/>
-                </material>
-            </visual>
-            <visual>
-                <origin xyz="0 ${-forearm_size_y * 0.36} ${forearm_size_z * 0.34}" rpy="0 0 0"/>
-                <geometry>
-                    <box size="${forearm_size_x * 0.82} ${forearm_rib_y} ${forearm_rib_z}"/>
-                </geometry>
-                <material name="arm_forearm_midline">
-                    <color rgba="0.34 0.38 0.45 1.0"/>
-                </material>
-            </visual>
-            <collision>
-                <origin xyz="0 0 0" rpy="0 0 0"/>
+                    <color rgba="0.25 0.30 0.35 1.0"/>
+                </material>
+            </visual>
+            <collision>
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