Commit message: Update face display URDF and body attachments

File: src/wall_climber/urdf/base_body.xacro (robot description, xacro)
@@ -1,159 +1,247 @@
 <?xml version="1.0"?>
 <robot xmlns:xacro="http://www.ros.org/wiki/xacro">
-    <xacro:macro name="base_body" params="">
-        <xacro:property name="robot_cfg" value="${xacro.load_yaml('$(find wall_climber)/config/cable_robot.yaml')}"/>
-        <xacro:property name="carriage_cfg" value="${robot_cfg['carriage']}"/>
-        <xacro:property name="attach_left_local_y" value="${-carriage_cfg['attachment_left_y']}"/>
-        <xacro:property name="attach_right_local_y" value="${-carriage_cfg['attachment_right_y']}"/>
-        <xacro:property name="mount_tip_z" value="${-(carriage_cfg['depth'] / 2.0) + 0.002}"/>
-        <xacro:property name="mount_sphere_radius" value="0.0050"/>
-        <xacro:property name="mount_sphere_highlight_radius" value="${mount_sphere_radius * 0.70}"/>
-        <xacro:property name="mount_stem_radius" value="0.0032"/>
-        <xacro:property name="mount_stem_length" value="0.006"/>
-        <xacro:property name="top_strip_width" value="${carriage_cfg['width'] - 0.050}"/>
-        <xacro:property name="top_strip_height" value="${carriage_cfg['height'] * 0.22}"/>
-        <xacro:property name="service_panel_width" value="${carriage_cfg['width'] * 0.18}"/>
-        <xacro:property name="service_panel_height" value="${carriage_cfg['height'] * 0.72}"/>
-        <xacro:property name="service_panel_x" value="${(carriage_cfg['width'] * 0.5) - (service_panel_width * 0.5) - 0.016}"/>
-        <xacro:property name="service_panel_y" value="${-(carriage_cfg['height'] * 0.13)}"/>
-        <link name="base_link">
-            <visual>
-                <geometry><box size="0.001 0.001 0.001"/></geometry>
-            </visual>
-            <inertial>
-                <mass value="0.01"/>
-                <inertia ixx="0.0001" ixy="0" ixz="0" iyy="0.0001" iyz="0" izz="0.0001"/>
-            </inertial>
-        </link>
-        <joint name="chassis_joint" type="fixed">
-            <parent link="base_link"/>
-            <child link="chassis"/>
-            <origin xyz="0 0 ${carriage_cfg['root_to_chassis_z']}" rpy="0 0 0"/>
-        </joint>
-        <link name="chassis">
-            <visual>
-                <origin xyz="0 0 0" rpy="0 0 0"/>
-                <geometry>
-                    <box size="${carriage_cfg['width']} ${carriage_cfg['height']} ${carriage_cfg['depth']}"/>
-                </geometry>
-                <material name="robot_orange_mat">
-                    <color rgba="1.0 0.35 0.05 1.0"/>
-                </material>
-            </visual>
-            <visual>
-                <origin xyz="-0.010 ${carriage_cfg['height'] * 0.27} ${carriage_cfg['depth'] * 0.05}" rpy="0 0 0"/>
-                <geometry>
-                    <box size="${top_strip_width} ${top_strip_height} ${carriage_cfg['depth'] * 0.32}"/>
-                </geometry>
-                <material name="robot_dark_top_trim">
-                    <color rgba="0.15 0.18 0.22 1.0"/>
-                </material>
-            </visual>
-            <visual>
-                <origin xyz="${service_panel_x} ${service_panel_y} ${carriage_cfg['depth'] * 0.08}" rpy="0 0 0"/>
-                <geometry>
-                    <box size="${service_panel_width} ${service_panel_height} ${carriage_cfg['depth'] * 0.28}"/>
-                </geometry>
-                <material name="robot_service_panel_mat">
-                    <color rgba="0.22 0.25 0.30 1.0"/>
-                </material>
-            </visual>
-            <visual>
-                <origin xyz="${service_panel_x} ${service_panel_y} ${carriage_cfg['depth'] * 0.20}" rpy="0 0 0"/>
-                <geometry>
-                    <box size="${service_panel_width * 0.72} ${service_panel_height * 0.52} ${carriage_cfg['depth'] * 0.08}"/>
-                </geometry>
-                <material name="robot_service_panel_highlight_mat">
-                    <color rgba="0.40 0.45 0.52 1.0"/>
-                </material>
-            </visual>
-            <collision>
-                <origin xyz="0 0 0" rpy="0 0 0"/>
-                <geometry>
-                    <box size="${carriage_cfg['width']} ${carriage_cfg['height']} ${carriage_cfg['depth']}"/>
-                </geometry>
-            </collision>
-            <inertial>
-                <origin xyz="0 0 0" rpy="0 0 0"/>
-                <mass value="${carriage_cfg['mass']}"/>
-                <inertia ixx="0.006" ixy="0.0" ixz="0.0" iyy="0.006" iyz="0.0" izz="0.006"/>
-            </inertial>
-        </link>
-        <joint name="left_cable_mount_joint" type="fixed">
-            <parent link="chassis"/>
-            <child link="left_cable_mount"/>
-            <origin xyz="${carriage_cfg['attachment_left_x']} ${attach_left_local_y} ${mount_tip_z}" rpy="0 0 0"/>
-        </joint>
-        <link name="left_cable_mount">
-            <visual>
-                <geometry><sphere radius="${mount_sphere_radius}"/></geometry>
-                <material name="cable_mount_ball_mat">
-                    <color rgba="0.86 0.10 0.10 1.0"/>
-                </material>
-            </visual>
-            <visual>
-                <origin xyz="0 0 0.0007" rpy="0 0 0"/>
-                <geometry><sphere radius="${mount_sphere_highlight_radius}"/></geometry>
-                <material name="cable_mount_ball_highlight_mat">
-                    <color rgba="1.0 0.34 0.30 1.0"/>
-                </material>
-            </visual>
-            <visual>
-                <origin xyz="0 0 ${mount_stem_length / 2.0}" rpy="0 0 0"/>
-                <geometry><cylinder radius="${mount_stem_radius}" length="${mount_stem_length}"/></geometry>
-                <material name="robot_dark_grey_mat">
-                    <color rgba="0.20 0.22 0.26 1.0"/>
-                </material>
-            </visual>
-            <collision>
-                <geometry><sphere radius="${mount_sphere_radius}"/></geometry>
-            </collision>
-            <collision>
-                <origin xyz="0 0 ${mount_stem_length / 2.0}" rpy="0 0 0"/>
-                <geometry><cylinder radius="${mount_stem_radius}" length="${mount_stem_length}"/></geometry>
-            </collision>
-            <inertial>
-                <mass value="0.015"/>
-                <inertia ixx="1.4e-5" ixy="0.0" ixz="0.0" iyy="1.4e-5" iyz="0.0" izz="1.4e-5"/>
-            </inertial>
-        </link>
-        <joint name="right_cable_mount_joint" type="fixed">
-            <parent link="chassis"/>
-            <child link="right_cable_mount"/>
-            <origin xyz="${carriage_cfg['attachment_right_x']} ${attach_right_local_y} ${mount_tip_z}" rpy="0 0 0"/>
-        </joint>
-        <link name="right_cable_mount">
-            <visual>
-                <geometry><sphere radius="${mount_sphere_radius}"/></geometry>
-                <material name="cable_mount_ball_mat">
-                    <color rgba="0.86 0.10 0.10 1.0"/>
-                </material>
-            </visual>
-            <visual>
-                <origin xyz="0 0 0.0007" rpy="0 0 0"/>
-                <geometry><sphere radius="${mount_sphere_highlight_radius}"/></geometry>
-                <material name="cable_mount_ball_highlight_mat">
-                    <color rgba="1.0 0.34 0.30 1.0"/>
-                </material>
-            </visual>
-            <visual>
-                <origin xyz="0 0 ${mount_stem_length / 2.0}" rpy="0 0 0"/>
-                <geometry><cylinder radius="${mount_stem_radius}" length="${mount_stem_length}"/></geometry>
-                <material name="robot_dark_grey_mat">
-                    <color rgba="0.20 0.22 0.26 1.0"/>
-                </material>
-            </visual>
-            <collision>
-                <geometry><sphere radius="${mount_sphere_radius}"/></geometry>
-            </collision>
-            <collision>
-                <origin xyz="0 0 ${mount_stem_length / 2.0}" rpy="0 0 0"/>
-                <geometry><cylinder radius="${mount_stem_radius}" length="${mount_stem_length}"/></geometry>
-            </collision>
-            <inertial>
-                <mass value="0.015"/>
-                <inertia ixx="1.4e-5" ixy="0.0" ixz="0.0" iyy="1.4e-5" iyz="0.0" izz="1.4e-5"/>
-            </inertial>
-        </link>
-    </xacro:macro>
+  <xacro:macro name="rounded_panel" params="x y z width height depth radius mat_name rgba">
+    <visual>
+      <origin xyz="${x} ${y} ${z}" rpy="0 0 0"/>
+      <geometry>
+        <box size="${width - 2.0 * radius} ${height} ${depth}"/>
+      </geometry>
+      <material name="${mat_name}">
+        <color rgba="${rgba}"/>
+      </material>
+    </visual>
+    <visual>
+      <origin xyz="${x} ${y} ${z}" rpy="0 0 0"/>
+      <geometry>
+        <box size="${width} ${height - 2.0 * radius} ${depth}"/>
+      </geometry>
+      <material name="${mat_name}">
+        <color rgba="${rgba}"/>
+      </material>
+    </visual>
+    <visual>
+      <origin xyz="${x - width / 2.0 + radius} ${y - height / 2.0 + radius} ${z}" rpy="0 0 0"/>
+      <geometry>
+        <cylinder radius="${radius}" length="${depth}"/>
+      </geometry>
+      <material name="${mat_name}">
+        <color rgba="${rgba}"/>
+      </material>
+    </visual>
+    <visual>
+      <origin xyz="${x + width / 2.0 - radius} ${y - height / 2.0 + radius} ${z}" rpy="0 0 0"/>
+      <geometry>
+        <cylinder radius="${radius}" length="${depth}"/>
+      </geometry>
+      <material name="${mat_name}">
+        <color rgba="${rgba}"/>
+      </material>
+    </visual>
+    <visual>
+      <origin xyz="${x - width / 2.0 + radius} ${y + height / 2.0 - radius} ${z}" rpy="0 0 0"/>
+      <geometry>
+        <cylinder radius="${radius}" length="${depth}"/>
+      </geometry>
+      <material name="${mat_name}">
+        <color rgba="${rgba}"/>
+      </material>
+    </visual>
+    <visual>
+      <origin xyz="${x + width / 2.0 - radius} ${y + height / 2.0 - radius} ${z}" rpy="0 0 0"/>
+      <geometry>
+        <cylinder radius="${radius}" length="${depth}"/>
+      </geometry>
+      <material name="${mat_name}">
+        <color rgba="${rgba}"/>
+      </material>
+    </visual>
+  </xacro:macro>
+  <xacro:macro name="body_cable_mount" params="link_name">
+    <link name="${link_name}">
+      <visual>
+        <origin xyz="0 0 0" rpy="0 0 0"/>
+        <geometry>
+          <cylinder radius="0.0046" length="0.0032"/>
+        </geometry>
+        <material name="${link_name}_head_mat">
+          <color rgba="0.72 0.75 0.80 1.0"/>
+        </material>
+      </visual>
+      <visual>
+        <origin xyz="0 0 0.0030" rpy="0 0 0"/>
+        <geometry>
+          <cylinder radius="0.0023" length="0.0060"/>
+        </geometry>
+        <material name="${link_name}_neck_mat">
+          <color rgba="0.18 0.20 0.24 1.0"/>
+        </material>
+      </visual>
+      <visual>
+        <origin xyz="0 0 0.0064" rpy="0 0 0"/>
+        <geometry>
+          <cylinder radius="0.0057" length="0.0028"/>
+        </geometry>
+        <material name="${link_name}_base_mat">
+          <color rgba="0.14 0.16 0.19 1.0"/>
+        </material>
+      </visual>
+      <visual>
+        <origin xyz="0 0 0.0079" rpy="0 0 0"/>
+        <geometry>
+          <box size="0.011 0.007 0.0032"/>
+        </geometry>
+        <material name="${link_name}_pad_mat">
+          <color rgba="0.22 0.25 0.29 1.0"/>
+        </material>
+      </visual>
+      <collision>
+        <origin xyz="0 0 0.0034" rpy="0 0 0"/>
+        <geometry>
+          <cylinder radius="0.0058" length="0.0105"/>
+        </geometry>
+      </collision>
+      <inertial>
+        <mass value="0.015"/>
+        <inertia ixx="1.4e-5" ixy="0.0" ixz="0.0" iyy="1.4e-5" iyz="0.0" izz="1.4e-5"/>
+      </inertial>
+    </link>
+  </xacro:macro>
+  <xacro:macro name="base_body" params="">
+    <xacro:property name="robot_cfg" value="${xacro.load_yaml('$(find wall_climber)/config/cable_robot.yaml')}"/>
+    <xacro:property name="carriage_cfg" value="${robot_cfg['carriage']}"/>
+    <xacro:property name="attach_left_local_y" value="${-carriage_cfg['attachment_left_y']}"/>
+    <xacro:property name="attach_right_local_y" value="${-carriage_cfg['attachment_right_y']}"/>
+    <xacro:property name="mount_tip_z" value="${-(carriage_cfg['depth'] / 2.0) + 0.002}"/>
+    <xacro:property name="front_mask_w" value="${carriage_cfg['width'] - 0.020}"/>
+    <xacro:property name="front_mask_h" value="${carriage_cfg['height'] - 0.018}"/>
+    <xacro:property name="front_mask_d" value="${carriage_cfg['depth'] * 0.18}"/>
+    <xacro:property name="front_mask_r" value="0.014"/>
+    <xacro:property name="front_mask_z" value="${carriage_cfg['depth'] / 2.0 - front_mask_d / 2.0 - 0.0005}"/>
+    <xacro:property name="top_band_w" value="${front_mask_w * 0.72}"/>
+    <xacro:property name="top_band_h" value="${carriage_cfg['height'] * 0.12}"/>
+    <xacro:property name="top_band_d" value="${carriage_cfg['depth'] * 0.10}"/>
+    <xacro:property name="top_band_z" value="${carriage_cfg['depth'] / 2.0 - top_band_d / 2.0 - 0.0002}"/>
+    <xacro:property name="chin_band_w" value="${front_mask_w * 0.78}"/>
+    <xacro:property name="chin_band_h" value="${carriage_cfg['height'] * 0.10}"/>
+    <xacro:property name="chin_band_d" value="${carriage_cfg['depth'] * 0.09}"/>
+    <xacro:property name="chin_band_z" value="${carriage_cfg['depth'] / 2.0 - chin_band_d / 2.0}"/>
+    <xacro:property name="side_rail_w" value="${carriage_cfg['width'] * 0.075}"/>
+    <xacro:property name="side_rail_h" value="${carriage_cfg['height'] * 0.64}"/>
+    <xacro:property name="side_rail_d" value="${carriage_cfg['depth'] * 0.09}"/>
+    <xacro:property name="side_rail_z" value="${carriage_cfg['depth'] / 2.0 - side_rail_d / 2.0}"/>
+    <xacro:property name="service_panel_w" value="${carriage_cfg['width'] * 0.15}"/>
+    <xacro:property name="service_panel_h" value="${carriage_cfg['height'] * 0.46}"/>
+    <xacro:property name="service_panel_d" value="${carriage_cfg['depth'] * 0.10}"/>
+    <xacro:property name="service_panel_x" value="${carriage_cfg['width'] * 0.28}"/>
+    <xacro:property name="service_panel_y" value="${-carriage_cfg['height'] * 0.04}"/>
+    <xacro:property name="service_panel_z" value="${carriage_cfg['depth'] / 2.0 - service_panel_d / 2.0}"/>
+    <link name="base_link">
+      <visual>
+        <geometry>
+          <box size="0.001 0.001 0.001"/>
+        </geometry>
+      </visual>
+      <inertial>
+        <mass value="0.01"/>
+        <inertia ixx="0.0001" ixy="0" ixz="0" iyy="0.0001" iyz="0" izz="0.0001"/>
+      </inertial>
+    </link>
+    <joint name="chassis_joint" type="fixed">
+      <parent link="base_link"/>
+      <child link="chassis"/>
+      <origin xyz="0 0 ${carriage_cfg['root_to_chassis_z']}" rpy="0 0 0"/>
+    </joint>
+    <link name="chassis">
+      <visual>
+        <origin xyz="0 0 0" rpy="0 0 0"/>
+        <geometry>
+          <box size="${carriage_cfg['width']} ${carriage_cfg['height']} ${carriage_cfg['depth']}"/>
+        </geometry>
+        <material name="robot_orange_shell_mat">
+          <color rgba="0.97 0.36 0.08 1.0"/>
+        </material>
+      </visual>
+      <xacro:rounded_panel
+        x="0" y="0" z="${front_mask_z}"
+        width="${front_mask_w}" height="${front_mask_h}" depth="${front_mask_d}" radius="${front_mask_r}"
+        mat_name="robot_front_mask_mat" rgba="0.12 0.14 0.17 1.0"/>
+      <visual>
+        <origin xyz="0 ${carriage_cfg['height'] * 0.33} ${top_band_z}" rpy="0 0 0"/>
+        <geometry>
+          <box size="${top_band_w} ${top_band_h} ${top_band_d}"/>
+        </geometry>
+        <material name="robot_top_band_mat">
+          <color rgba="0.20 0.23 0.28 1.0"/>
+        </material>
+      </visual>
+      <visual>
+        <origin xyz="0 ${-carriage_cfg['height'] * 0.35} ${chin_band_z}" rpy="0 0 0"/>
+        <geometry>
+          <box size="${chin_band_w} ${chin_band_h} ${chin_band_d}"/>
+        </geometry>
+        <material name="robot_chin_band_mat">
+          <color rgba="0.18 0.21 0.25 1.0"/>
+        </material>
+      </visual>
+      <visual>
+        <origin xyz="${-(carriage_cfg['width'] * 0.5) + (side_rail_w * 0.5) + 0.008} 0 ${side_rail_z}" rpy="0 0 0"/>
+        <geometry>
+          <box size="${side_rail_w} ${side_rail_h} ${side_rail_d}"/>
+        </geometry>
+        <material name="robot_side_rail_mat">
+          <color rgba="0.22 0.25 0.30 1.0"/>
+        </material>
+      </visual>
+      <visual>
+        <origin xyz="${(carriage_cfg['width'] * 0.5) - (side_rail_w * 0.5) - 0.008} 0 ${side_rail_z}" rpy="0 0 0"/>
+        <geometry>
+          <box size="${side_rail_w} ${side_rail_h} ${side_rail_d}"/>
+        </geometry>
+        <material name="robot_side_rail_mat">
+          <color rgba="0.22 0.25 0.30 1.0"/>
+        </material>
+      </visual>
+      <visual>
+        <origin xyz="${service_panel_x} ${service_panel_y} ${service_panel_z}" rpy="0 0 0"/>
+        <geometry>
+          <box size="${service_panel_w} ${service_panel_h} ${service_panel_d}"/>
+        </geometry>
+        <material name="robot_service_panel_mat">
+          <color rgba="0.21 0.24 0.28 1.0"/>
+        </material>
+      </visual>
+      <visual>
+        <origin xyz="${service_panel_x} ${service_panel_y} ${service_panel_z + 0.0015}" rpy="0 0 0"/>
+        <geometry>
+          <box size="${service_panel_w * 0.72} ${service_panel_h * 0.55} ${service_panel_d * 0.36}"/>
+        </geometry>
+        <material name="robot_service_inset_mat">
+          <color rgba="0.44 0.48 0.54 1.0"/>
+        </material>
+      </visual>
+      <collision>
+        <origin xyz="0 0 0" rpy="0 0 0"/>
+        <geometry>
+          <box size="${carriage_cfg['width']} ${carriage_cfg['height']} ${carriage_cfg['depth']}"/>
+        </geometry>
+      </collision>
+      <inertial>
+        <origin xyz="0 0 0" rpy="0 0 0"/>
+        <mass value="${carriage_cfg['mass']}"/>
+        <inertia ixx="0.006" ixy="0.0" ixz="0.0" iyy="0.006" iyz="0.0" izz="0.006"/>
+      </inertial>
+    </link>
+    <joint name="left_cable_mount_joint" type="fixed">
+      <parent link="chassis"/>
+      <child link="left_cable_mount"/>
+      <origin xyz="${carriage_cfg['attachment_left_x']} ${attach_left_local_y} ${mount_tip_z}" rpy="0 0 0"/>
+    </joint>
+    <xacro:body_cable_mount link_name="left_cable_mount"/>
+    <joint name="right_cable_mount_joint" type="fixed">
+      <parent link="chassis"/>
+      <child link="right_cable_mount"/>
+      <origin xyz="${carriage_cfg['attachment_right_x']} ${attach_right_local_y} ${mount_tip_z}" rpy="0 0 0"/>
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
File: src/wall_climber/urdf/cable_supervisor.urdf.xacro (robot description, xacro)
@@ -16,5 +16,62 @@
   <xacro:property name="cable_mount_right_local_y" value="${-carriage_cfg['attachment_right_y']}"/>
   <xacro:property name="cable_mount_local_z" value="${chassis_root_local_z - (carriage_cfg['depth'] / 2.0) + 0.002}"/>
+  <xacro:property name="board_left_world_x" value="${board_cfg['center_x'] - (board_cfg['width'] / 2.0)}"/>
+  <xacro:property name="board_top_world_z" value="${board_cfg['center_z'] + (board_cfg['height'] / 2.0)}"/>
+  <xacro:property name="left_anchor_world_x" value="${board_left_world_x + anchor_cfg['left_x']}"/>
+  <xacro:property name="left_anchor_world_z" value="${board_top_world_z - anchor_cfg['left_y']}"/>
+  <xacro:property name="right_anchor_world_x" value="${board_left_world_x + anchor_cfg['right_x']}"/>
+  <xacro:property name="right_anchor_world_z" value="${board_top_world_z - anchor_cfg['right_y']}"/>
+  <xacro:macro name="board_anchor_visual" params="name world_x world_z x_sign">
+    <joint name="${name}_joint" type="fixed">
+      <parent link="base_link"/>
+      <child link="${name}"/>
+      <origin xyz="${world_x} ${board_cfg['surface_y']} ${world_z}" rpy="0 0 0"/>
+    </joint>
+    <link name="${name}">
+      <visual>
+        <origin xyz="${0.016 * x_sign} 0.014 -0.016" rpy="0 0 0"/>
+        <geometry>
+          <box size="0.036 0.006 0.036"/>
+        </geometry>
+        <material name="${name}_plate_mat">
+          <color rgba="0.14 0.16 0.19 1.0"/>
+        </material>
+      </visual>
+      <visual>
+        <origin xyz="${0.010 * x_sign} 0.008 -0.010" rpy="0 0 0"/>
+        <geometry>
+          <box size="0.020 0.012 0.020"/>
+        </geometry>
+        <material name="${name}_body_mat">
+          <color rgba="0.22 0.25 0.30 1.0"/>
+        </material>
+      </visual>
+      <visual>
+        <origin xyz="0 0 0" rpy="1.57079632679 0 0"/>
+        <geometry>
+          <cylinder radius="0.0095" length="0.010"/>
+        </geometry>
+        <material name="${name}_roller_mat">
+          <color rgba="0.74 0.77 0.82 1.0"/>
+        </material>
+      </visual>
+      <visual>
+        <origin xyz="0 0 0" rpy="1.57079632679 0 0"/>
+        <geometry>
+          <cylinder radius="0.0022" length="0.015"/>
+        </geometry>
+        <material name="${name}_axle_mat">
+          <color rgba="0.18 0.20 0.24 1.0"/>
+        </material>
+      </visual>
+      <inertial>
+        <mass value="0.04"/>
+        <inertia ixx="2.0e-5" ixy="0.0" ixz="0.0" iyy="2.0e-5" iyz="0.0" izz="2.0e-5"/>
+      </inertial>
+    </link>
+  </xacro:macro>
   <link name="base_link"/>
+  <xacro:board_anchor_visual name="left_board_anchor" world_x="${left_anchor_world_x}" world_z="${left_anchor_world_z}" x_sign="1"/>
+  <xacro:board_anchor_visual name="right_board_anchor" world_x="${right_anchor_world_x}" world_z="${right_anchor_world_z}" x_sign="-1"/>
   <webots>
     <plugin type="wall_climber.cable_supervisor_plugin.CableSupervisorPlugin">
