Commit message: Update face display URDF and body attachments

File: src/wall_climber/urdf/robot_face_screen.xacro (robot description, xacro)
@@ -1,51 +1,141 @@
 <?xml version="1.0"?>
 <robot xmlns:xacro="http://www.ros.org/wiki/xacro">
-        <xacro:macro name="robot_face_screen" params="">
-        <xacro:property name="robot_cfg" value="${xacro.load_yaml('$(find wall_climber)/config/cable_robot.yaml')}"/>
-        <xacro:property name="carriage_cfg" value="${robot_cfg['carriage']}"/>
-        <xacro:property name="face_width" value="${carriage_cfg['width'] - 0.034}"/>
-        <xacro:property name="face_height" value="${carriage_cfg['height'] - 0.032}"/>
-        <xacro:property name="screen_width" value="${face_width - 0.030}"/>
-        <xacro:property name="screen_height" value="${face_height - 0.026}"/>
-        <joint name="face_joint" type="fixed">
-            <parent link="chassis"/>
-            <child link="face_link"/>
-            <origin xyz="-0.014 -0.003 ${carriage_cfg['depth'] / 2.0 + 0.001}" rpy="0 0 0"/>
-        </joint>
-        <link name="face_link">
-            <visual>
-                <geometry> <box size="${face_width} ${face_height} 0.01"/> </geometry>
-                <material name="face_black">
-                    <color rgba="0.06 0.06 0.06 1.0"/>
-                </material>
-            </visual>
-            <collision>
-                <geometry> <box size="${face_width} ${face_height} 0.01"/> </geometry>
-            </collision>
-            <inertial>
-                <mass value="0.05"/>
-                <inertia ixx="0.0001" ixy="0" ixz="0" iyy="0.0001" iyz="0" izz="0.0001"/>
-            </inertial>
-        </link>
-        <joint name="screen_joint" type="fixed">
-            <parent link="face_link"/>
-            <child link="screen_link"/>
-            <origin xyz="0 0 0.006" rpy="0 0 0"/>
-        </joint>
-        <link name="screen_link">
-            <visual>
-                <geometry> <box size="${screen_width} ${screen_height} 0.002"/> </geometry>
-                <material name="screen_cyan">
-                    <color rgba="0.05 0.95 1.0 1.0"/>
-                </material>
-            </visual>
-            <collision>
-                <geometry> <box size="${screen_width} ${screen_height} 0.002"/> </geometry>
-            </collision>
-            <inertial>
-                <mass value="0.02"/>
-                <inertia ixx="0.00001" ixy="0" ixz="0" iyy="0.00001" iyz="0" izz="0.00001"/>
-            </inertial>
-        </link>
-    </xacro:macro>
+  <xacro:macro name="rounded_panel" params="x y z width height depth radius mat_name rgba">
+    <visual>
+      <origin xyz="${x} ${y} ${z}" rpy="0 0 0"/>
+      <geometry>
+        <box size="${width - 2.0 * radius} ${height} ${depth}"/>
+      </geometry>
+      <material name="${mat_name}">
+        <color rgba="${rgba}"/>
+      </material>
+    </visual>
+    <visual>
+      <origin xyz="${x} ${y} ${z}" rpy="0 0 0"/>
+      <geometry>
+        <box size="${width} ${height - 2.0 * radius} ${depth}"/>
+      </geometry>
+      <material name="${mat_name}">
+        <color rgba="${rgba}"/>
+      </material>
+    </visual>
+    <visual>
+      <origin xyz="${x - width / 2.0 + radius} ${y - height / 2.0 + radius} ${z}" rpy="0 0 0"/>
+      <geometry>
+        <cylinder radius="${radius}" length="${depth}"/>
+      </geometry>
+      <material name="${mat_name}">
+        <color rgba="${rgba}"/>
+      </material>
+    </visual>
+    <visual>
+      <origin xyz="${x + width / 2.0 - radius} ${y - height / 2.0 + radius} ${z}" rpy="0 0 0"/>
+      <geometry>
+        <cylinder radius="${radius}" length="${depth}"/>
+      </geometry>
+      <material name="${mat_name}">
+        <color rgba="${rgba}"/>
+      </material>
+    </visual>
+    <visual>
+      <origin xyz="${x - width / 2.0 + radius} ${y + height / 2.0 - radius} ${z}" rpy="0 0 0"/>
+      <geometry>
+        <cylinder radius="${radius}" length="${depth}"/>
+      </geometry>
+      <material name="${mat_name}">
+        <color rgba="${rgba}"/>
+      </material>
+    </visual>
+    <visual>
+      <origin xyz="${x + width / 2.0 - radius} ${y + height / 2.0 - radius} ${z}" rpy="0 0 0"/>
+      <geometry>
+        <cylinder radius="${radius}" length="${depth}"/>
+      </geometry>
+      <material name="${mat_name}">
+        <color rgba="${rgba}"/>
+      </material>
+    </visual>
+  </xacro:macro>
+  <xacro:macro name="robot_face_screen" params="">
+    <xacro:property name="robot_cfg" value="${xacro.load_yaml('$(find wall_climber)/config/cable_robot.yaml')}"/>
+    <xacro:property name="carriage_cfg" value="${robot_cfg['carriage']}"/>
+    <xacro:property name="face_width" value="${carriage_cfg['width'] - 0.030}"/>
+    <xacro:property name="face_height" value="${carriage_cfg['height'] - 0.028}"/>
+    <xacro:property name="face_depth" value="0.010"/>
+    <xacro:property name="face_radius" value="0.012"/>
+    <xacro:property name="bezel_width" value="${face_width - 0.014}"/>
+    <xacro:property name="bezel_height" value="${face_height - 0.016}"/>
+    <xacro:property name="bezel_depth" value="0.0040"/>
+    <xacro:property name="bezel_radius" value="0.010"/>
+    <xacro:property name="screen_width" value="${bezel_width - 0.012}"/>
+    <xacro:property name="screen_height" value="${bezel_height - 0.012}"/>
+    <xacro:property name="screen_depth" value="0.0022"/>
+    <xacro:property name="screen_radius" value="0.008"/>
+    <joint name="face_joint" type="fixed">
+      <parent link="chassis"/>
+      <child link="face_link"/>
+      <origin xyz="-0.006 0.0 ${carriage_cfg['depth'] / 2.0 + face_depth / 2.0 + 0.001}" rpy="0 0 0"/>
+    </joint>
+    <link name="face_link">
+      <xacro:rounded_panel
+        x="0" y="0" z="0"
+        width="${face_width}" height="${face_height}" depth="${face_depth}" radius="${face_radius}"
+        mat_name="face_outer_shell_mat" rgba="0.08 0.09 0.11 1.0"/>
+      <visual>
+        <origin xyz="0 ${face_height * 0.34} ${face_depth * 0.18}" rpy="0 0 0"/>
+        <geometry>
+          <box size="${face_width * 0.72} ${face_height * 0.10} 0.006"/>
+        </geometry>
+        <material name="face_brow_bar_mat">
+          <color rgba="0.18 0.21 0.26 1.0"/>
+        </material>
+      </visual>
+      <visual>
+        <origin xyz="0 ${-face_height * 0.36} ${face_depth * 0.14}" rpy="0 0 0"/>
+        <geometry>
+          <box size="${face_width * 0.66} ${face_height * 0.08} 0.005"/>
+        </geometry>
+        <material name="face_chin_bar_mat">
+          <color rgba="0.18 0.21 0.25 1.0"/>
+        </material>
+      </visual>
+      <collision>
+        <geometry>
+          <box size="${face_width} ${face_height} ${face_depth}"/>
+        </geometry>
+      </collision>
+      <inertial>
+        <mass value="0.05"/>
+        <inertia ixx="0.0001" ixy="0" ixz="0" iyy="0.0001" iyz="0" izz="0.0001"/>
+      </inertial>
+    </link>
+    <joint name="screen_joint" type="fixed">
+      <parent link="face_link"/>
+      <child link="screen_link"/>
+      <origin xyz="0 0 ${face_depth / 2.0 + bezel_depth / 2.0 + 0.0008}" rpy="0 0 0"/>
+    </joint>
+    <link name="screen_link">
+      <xacro:rounded_panel
+        x="0" y="0" z="0"
+        width="${bezel_width}" height="${bezel_height}" depth="${bezel_depth}" radius="${bezel_radius}"
+        mat_name="screen_bezel_mat" rgba="0.02 0.03 0.04 1.0"/>
+      <xacro:rounded_panel
+        x="0" y="0" z="${bezel_depth / 2.0 + screen_depth / 2.0 - 0.0004}"
+        width="${screen_width}" height="${screen_height}" depth="${screen_depth}" radius="${screen_radius}"
+        mat_name="screen_glass_mat" rgba="0.03 0.10 0.14 1.0"/>
+      <xacro:rounded_panel
+        x="0" y="0" z="${bezel_depth / 2.0 + screen_depth + 0.0002}"
+        width="${screen_width * 0.96}" height="${screen_height * 0.96}" depth="0.0008" radius="${screen_radius * 0.92}"
+        mat_name="screen_emit_mat" rgba="0.05 0.84 0.92 1.0"/>
+      <collision>
+        <geometry>
+          <box size="${bezel_width} ${bezel_height} ${bezel_depth}"/>
+        </geometry>
+      </collision>
+      <inertial>
+        <mass value="0.02"/>
+        <inertia ixx="0.00001" ixy="0" ixz="0" iyy="0.00001" iyz="0" izz="0.00001"/>
+      </inertial>
+    </link>
+  </xacro:macro>
 </robot>
