Commit message: Complete visual updates and face display wiring

File: src/wall_climber/urdf/base_body.xacro (robot description, xacro)
@@ -133,7 +133,27 @@
     <xacro:property name="service_panel_h" value="${carriage_cfg['height'] * 0.46}"/>
     <xacro:property name="service_panel_d" value="${carriage_cfg['depth'] * 0.10}"/>
-    <xacro:property name="service_panel_x" value="${carriage_cfg['width'] * 0.28}"/>
+    <xacro:property name="service_panel_x" value="${-carriage_cfg['width'] * 0.28}"/>
     <xacro:property name="service_panel_y" value="${-carriage_cfg['height'] * 0.04}"/>
     <xacro:property name="service_panel_z" value="${carriage_cfg['depth'] / 2.0 - service_panel_d / 2.0}"/>
+    <xacro:property name="arm_exit_slot_x" value="${(carriage_cfg['width'] * 0.5) - ((carriage_cfg['width'] * 0.18) * 0.5) - 0.016}"/>
+    <xacro:property name="arm_exit_slot_y" value="${-carriage_cfg['pen_offset_y']}"/>
+    <xacro:property name="arm_exit_slot_w" value="${carriage_cfg['width'] * 0.26}"/>
+    <xacro:property name="arm_exit_slot_h" value="${carriage_cfg['height'] * 0.48}"/>
+    <xacro:property name="arm_exit_slot_d" value="${carriage_cfg['depth'] * 0.08}"/>
+    <xacro:property name="arm_exit_slot_z" value="${-(carriage_cfg['depth'] / 2.0) + arm_exit_slot_d / 2.0 + 0.0004}"/>
+    <xacro:property name="arm_exit_bezel_t" value="0.006"/>
+    <xacro:property name="arm_exit_bezel_d" value="${carriage_cfg['depth'] * 0.07}"/>
+    <xacro:property name="arm_exit_bezel_z" value="${-(carriage_cfg['depth'] / 2.0) + arm_exit_bezel_d / 2.0 + 0.0008}"/>
+    <xacro:property name="arm_exit_rail_w" value="${arm_exit_slot_w * 0.72}"/>
+    <xacro:property name="arm_exit_rail_h" value="0.0036"/>
+    <xacro:property name="arm_exit_rail_d" value="${carriage_cfg['depth'] * 0.09}"/>
+    <xacro:property name="arm_exit_rail_z" value="${-(carriage_cfg['depth'] / 2.0) + arm_exit_rail_d / 2.0 + 0.0012}"/>
+    <xacro:property name="vent_slit_w" value="${service_panel_w * 0.68}"/>
+    <xacro:property name="vent_slit_h" value="0.0040"/>
+    <xacro:property name="vent_slit_d" value="${service_panel_d * 0.48}"/>
+    <xacro:property name="vent_slit_z" value="${service_panel_z + service_panel_d * 0.32}"/>
+    <xacro:property name="accent_bolt_r" value="0.0031"/>
+    <xacro:property name="accent_bolt_l" value="0.0028"/>
+    <xacro:property name="accent_bolt_z" value="${carriage_cfg['depth'] / 2.0 + accent_bolt_l / 2.0 + 0.0006}"/>
     <link name="base_link">
       <visual>
@@ -219,4 +239,123 @@
           <color rgba="0.44 0.48 0.54 1.0"/>
         </material>
+      </visual>
+      <visual>
+        <origin xyz="${service_panel_x} ${service_panel_y + service_panel_h * 0.22} ${vent_slit_z}" rpy="0 0 0"/>
+        <geometry>
+          <box size="${vent_slit_w} ${vent_slit_h} ${vent_slit_d}"/>
+        </geometry>
+        <material name="robot_vent_slat_mat">
+          <color rgba="0.09 0.10 0.12 1.0"/>
+        </material>
+      </visual>
+      <visual>
+        <origin xyz="${service_panel_x} ${service_panel_y + service_panel_h * 0.10} ${vent_slit_z}" rpy="0 0 0"/>
+        <geometry>
+          <box size="${vent_slit_w} ${vent_slit_h} ${vent_slit_d}"/>
+        </geometry>
+        <material name="robot_vent_slat_mat">
+          <color rgba="0.09 0.10 0.12 1.0"/>
+        </material>
+      </visual>
+      <visual>
+        <origin xyz="${service_panel_x} ${service_panel_y - service_panel_h * 0.02} ${vent_slit_z}" rpy="0 0 0"/>
+        <geometry>
+          <box size="${vent_slit_w} ${vent_slit_h} ${vent_slit_d}"/>
+        </geometry>
+        <material name="robot_vent_slat_mat">
+          <color rgba="0.09 0.10 0.12 1.0"/>
+        </material>
+      </visual>
+      <visual>
+        <origin xyz="${service_panel_x} ${service_panel_y - service_panel_h * 0.14} ${vent_slit_z}" rpy="0 0 0"/>
+        <geometry>
+          <box size="${vent_slit_w} ${vent_slit_h} ${vent_slit_d}"/>
+        </geometry>
+        <material name="robot_vent_slat_mat">
+          <color rgba="0.09 0.10 0.12 1.0"/>
+        </material>
+      </visual>
+      <visual>
+        <origin xyz="${arm_exit_slot_x} ${arm_exit_slot_y} ${arm_exit_slot_z}" rpy="0 0 0"/>
+        <geometry>
+          <box size="${arm_exit_slot_w} ${arm_exit_slot_h} ${arm_exit_slot_d}"/>
+        </geometry>
+        <material name="robot_arm_exit_recess_mat">
+          <color rgba="0.025 0.027 0.032 1.0"/>
+        </material>
+      </visual>
+      <visual>
+        <origin xyz="${arm_exit_slot_x} ${arm_exit_slot_y + arm_exit_slot_h / 2.0 + arm_exit_bezel_t / 2.0} ${arm_exit_bezel_z}" rpy="0 0 0"/>
+        <geometry>
+          <box size="${arm_exit_slot_w + 2.0 * arm_exit_bezel_t} ${arm_exit_bezel_t} ${arm_exit_bezel_d}"/>
+        </geometry>
+        <material name="robot_arm_exit_bezel_mat">
+          <color rgba="0.20 0.23 0.28 1.0"/>
+        </material>
+      </visual>
+      <visual>
+        <origin xyz="${arm_exit_slot_x} ${arm_exit_slot_y - arm_exit_slot_h / 2.0 - arm_exit_bezel_t / 2.0} ${arm_exit_bezel_z}" rpy="0 0 0"/>
+        <geometry>
+          <box size="${arm_exit_slot_w + 2.0 * arm_exit_bezel_t} ${arm_exit_bezel_t} ${arm_exit_bezel_d}"/>
+        </geometry>
+        <material name="robot_arm_exit_bezel_mat">
+          <color rgba="0.20 0.23 0.28 1.0"/>
+        </material>
+      </visual>
+      <visual>
+        <origin xyz="${arm_exit_slot_x - arm_exit_slot_w / 2.0 - arm_exit_bezel_t / 2.0} ${arm_exit_slot_y} ${arm_exit_bezel_z}" rpy="0 0 0"/>
+        <geometry>
+          <box size="${arm_exit_bezel_t} ${arm_exit_slot_h + 2.0 * arm_exit_bezel_t} ${arm_exit_bezel_d}"/>
+        </geometry>
+        <material name="robot_arm_exit_bezel_mat">
+          <color rgba="0.20 0.23 0.28 1.0"/>
+        </material>
+      </visual>
+      <visual>
+        <origin xyz="${arm_exit_slot_x + arm_exit_slot_w / 2.0 + arm_exit_bezel_t / 2.0} ${arm_exit_slot_y} ${arm_exit_bezel_z}" rpy="0 0 0"/>
+        <geometry>
+          <box size="${arm_exit_bezel_t} ${arm_exit_slot_h + 2.0 * arm_exit_bezel_t} ${arm_exit_bezel_d}"/>
+        </geometry>
+        <material name="robot_arm_exit_bezel_mat">
+          <color rgba="0.20 0.23 0.28 1.0"/>
+        </material>
+      </visual>
+      <visual>
+        <origin xyz="${arm_exit_slot_x} ${arm_exit_slot_y + arm_exit_slot_h * 0.22} ${arm_exit_rail_z}" rpy="0 0 0"/>
+        <geometry>
+          <box size="${arm_exit_rail_w} ${arm_exit_rail_h} ${arm_exit_rail_d}"/>
+        </geometry>
+        <material name="robot_arm_exit_rail_mat">
+          <color rgba="0.54 0.58 0.64 1.0"/>
+        </material>
+      </visual>
+      <visual>
+        <origin xyz="${arm_exit_slot_x} ${arm_exit_slot_y - arm_exit_slot_h * 0.22} ${arm_exit_rail_z}" rpy="0 0 0"/>
+        <geometry>
+          <box size="${arm_exit_rail_w} ${arm_exit_rail_h} ${arm_exit_rail_d}"/>
+        </geometry>
+        <material name="robot_arm_exit_rail_mat">
+          <color rgba="0.54 0.58 0.64 1.0"/>
+        </material>
+      </visual>
+      <visual>
+        <origin xyz="${-front_mask_w / 2.0 + 0.018} ${front_mask_h / 2.0 - 0.018} ${accent_bolt_z}" rpy="0 0 0"/>
+        <geometry><cylinder radius="${accent_bolt_r}" length="${accent_bolt_l}"/></geometry>
+        <material name="robot_corner_bolt_mat"><color rgba="0.64 0.68 0.74 1.0"/></material>
+      </visual>
+      <visual>
+        <origin xyz="${front_mask_w / 2.0 - 0.018} ${front_mask_h / 2.0 - 0.018} ${accent_bolt_z}" rpy="0 0 0"/>
+        <geometry><cylinder radius="${accent_bolt_r}" length="${accent_bolt_l}"/></geometry>
+        <material name="robot_corner_bolt_mat"><color rgba="0.64 0.68 0.74 1.0"/></material>
+      </visual>
+      <visual>
+        <origin xyz="${-front_mask_w / 2.0 + 0.018} ${-front_mask_h / 2.0 + 0.018} ${accent_bolt_z}" rpy="0 0 0"/>
+        <geometry><cylinder radius="${accent_bolt_r}" length="${accent_bolt_l}"/></geometry>
+        <material name="robot_corner_bolt_mat"><color rgba="0.64 0.68 0.74 1.0"/></material>
+      </visual>
+      <visual>
+        <origin xyz="${front_mask_w / 2.0 - 0.018} ${-front_mask_h / 2.0 + 0.018} ${accent_bolt_z}" rpy="0 0 0"/>
+        <geometry><cylinder radius="${accent_bolt_r}" length="${accent_bolt_l}"/></geometry>
+        <material name="robot_corner_bolt_mat"><color rgba="0.64 0.68 0.74 1.0"/></material>
       </visual>
       <collision>

File: src/wall_climber/urdf/cable_supervisor.urdf.xacro (robot description, xacro)
@@ -26,5 +26,5 @@
   <xacro:property name="bottom_right_anchor_world_x" value="${board_left_world_x + anchor_cfg['bottom_right_x']}"/>
   <xacro:property name="bottom_right_anchor_world_z" value="${board_top_world_z - anchor_cfg['bottom_right_y']}"/>
-  <xacro:macro name="board_anchor_visual" params="name world_x world_z x_sign">
+  <xacro:macro name="board_anchor_visual" params="name world_x world_z x_sign z_sign">
     <joint name="${name}_joint" type="fixed">
       <parent link="base_link"/>
@@ -34,37 +34,93 @@
     <link name="${name}">
       <visual>
-        <origin xyz="${0.016 * x_sign} 0.014 -0.016" rpy="0 0 0"/>
-        <geometry>
-          <box size="0.036 0.006 0.036"/>
-        </geometry>
-        <material name="${name}_plate_mat">
-          <color rgba="0.14 0.16 0.19 1.0"/>
-        </material>
-      </visual>
-      <visual>
-        <origin xyz="${0.010 * x_sign} 0.008 -0.010" rpy="0 0 0"/>
-        <geometry>
-          <box size="0.020 0.012 0.020"/>
-        </geometry>
-        <material name="${name}_body_mat">
-          <color rgba="0.22 0.25 0.30 1.0"/>
-        </material>
-      </visual>
-      <visual>
-        <origin xyz="0 0 0" rpy="1.57079632679 0 0"/>
-        <geometry>
-          <cylinder radius="0.0095" length="0.010"/>
-        </geometry>
-        <material name="${name}_roller_mat">
-          <color rgba="0.74 0.77 0.82 1.0"/>
-        </material>
-      </visual>
-      <visual>
-        <origin xyz="0 0 0" rpy="1.57079632679 0 0"/>
-        <geometry>
-          <cylinder radius="0.0022" length="0.015"/>
-        </geometry>
-        <material name="${name}_axle_mat">
-          <color rgba="0.18 0.20 0.24 1.0"/>
+        <origin xyz="${0.018 * x_sign} 0.010 ${0.018 * z_sign}" rpy="0 0 0"/>
+        <geometry>
+          <box size="0.050 0.007 0.050"/>
+        </geometry>
+        <material name="${name}_mounting_plate_mat">
+          <color rgba="0.12 0.14 0.17 1.0"/>
+        </material>
+      </visual>
+      <visual>
+        <origin xyz="${0.018 * x_sign} 0.025 ${0.018 * z_sign}" rpy="0 0 0"/>
+        <geometry>
+          <box size="0.038 0.026 0.038"/>
+        </geometry>
+        <material name="${name}_motor_housing_mat">
+          <color rgba="0.23 0.26 0.31 1.0"/>
+        </material>
+      </visual>
+      <visual>
+        <origin xyz="${0.018 * x_sign} 0.040 ${0.018 * z_sign}" rpy="0 0 0"/>
+        <geometry>
+          <box size="0.041 0.0045 0.041"/>
+        </geometry>
+        <material name="${name}_accent_band_mat">
+          <color rgba="0.55 0.60 0.67 1.0"/>
+        </material>
+      </visual>
+      <visual>
+        <origin xyz="${0.041 * x_sign} 0.027 ${0.018 * z_sign}" rpy="0 0 0"/>
+        <geometry>
+          <box size="0.011 0.018 0.016"/>
+        </geometry>
+        <material name="${name}_connector_cap_mat">
+          <color rgba="0.08 0.09 0.11 1.0"/>
+        </material>
+      </visual>
+      <visual>
+        <origin xyz="${0.018 * x_sign - 0.013} 0.044 ${0.018 * z_sign - 0.013}" rpy="1.57079632679 0 0"/>
+        <geometry><cylinder radius="0.0028" length="0.004"/></geometry>
+        <material name="${name}_bolt_mat"><color rgba="0.70 0.74 0.80 1.0"/></material>
+      </visual>
+      <visual>
+        <origin xyz="${0.018 * x_sign + 0.013} 0.044 ${0.018 * z_sign - 0.013}" rpy="1.57079632679 0 0"/>
+        <geometry><cylinder radius="0.0028" length="0.004"/></geometry>
+        <material name="${name}_bolt_mat"><color rgba="0.70 0.74 0.80 1.0"/></material>
+      </visual>
+      <visual>
+        <origin xyz="${0.018 * x_sign - 0.013} 0.044 ${0.018 * z_sign + 0.013}" rpy="1.57079632679 0 0"/>
+        <geometry><cylinder radius="0.0028" length="0.004"/></geometry>
+        <material name="${name}_bolt_mat"><color rgba="0.70 0.74 0.80 1.0"/></material>
+      </visual>
+      <visual>
+        <origin xyz="${0.018 * x_sign + 0.013} 0.044 ${0.018 * z_sign + 0.013}" rpy="1.57079632679 0 0"/>
+        <geometry><cylinder radius="0.0028" length="0.004"/></geometry>
+        <material name="${name}_bolt_mat"><color rgba="0.70 0.74 0.80 1.0"/></material>
+      </visual>
+      <visual>
+        <origin xyz="0 0.043 0" rpy="1.57079632679 0 0"/>
+        <geometry>
+          <cylinder radius="0.0048" length="0.014"/>
+        </geometry>
+        <material name="${name}_output_shaft_mat">
+          <color rgba="0.72 0.75 0.80 1.0"/>
+        </material>
+      </visual>
+      <visual>
+        <origin xyz="0 0.052 0" rpy="1.57079632679 0 0"/>
+        <geometry>
+          <cylinder radius="0.0135" length="0.011"/>
+        </geometry>
+        <material name="${name}_pulley_mat">
+          <color rgba="0.36 0.39 0.44 1.0"/>
+        </material>
+      </visual>
+      <visual>
+        <origin xyz="0 0.052 0" rpy="1.57079632679 0 0"/>
+        <geometry>
+          <cylinder radius="0.0142" length="0.0022"/>
+        </geometry>
+        <material name="${name}_pulley_groove_mat">
+          <color rgba="0.08 0.09 0.11 1.0"/>
+        </material>
+      </visual>
+      <visual>
+        <origin xyz="0 0.059 0" rpy="1.57079632679 0 0"/>
+        <geometry>
+          <cylinder radius="0.0065" length="0.006"/>
+        </geometry>
+        <material name="${name}_pulley_hub_mat">
+          <color rgba="0.68 0.71 0.76 1.0"/>
         </material>
       </visual>
@@ -76,8 +132,8 @@
   </xacro:macro>
   <link name="base_link"/>
-  <xacro:board_anchor_visual name="left_board_anchor" world_x="${left_anchor_world_x}" world_z="${left_anchor_world_z}" x_sign="1"/>
-  <xacro:board_anchor_visual name="right_board_anchor" world_x="${right_anchor_world_x}" world_z="${right_anchor_world_z}" x_sign="-1"/>
-  <xacro:board_anchor_visual name="bottom_left_board_anchor" world_x="${bottom_left_anchor_world_x}" world_z="${bottom_left_anchor_world_z}" x_sign="1"/>
-  <xacro:board_anchor_visual name="bottom_right_board_anchor" world_x="${bottom_right_anchor_world_x}" world_z="${bottom_right_anchor_world_z}" x_sign="-1"/>
+  <xacro:board_anchor_visual name="left_board_anchor" world_x="${left_anchor_world_x}" world_z="${left_anchor_world_z}" x_sign="1" z_sign="-1"/>
+  <xacro:board_anchor_visual name="right_board_anchor" world_x="${right_anchor_world_x}" world_z="${right_anchor_world_z}" x_sign="-1" z_sign="-1"/>
+  <xacro:board_anchor_visual name="bottom_left_board_anchor" world_x="${bottom_left_anchor_world_x}" world_z="${bottom_left_anchor_world_z}" x_sign="1" z_sign="1"/>
+  <xacro:board_anchor_visual name="bottom_right_board_anchor" world_x="${bottom_right_anchor_world_x}" world_z="${bottom_right_anchor_world_z}" x_sign="-1" z_sign="1"/>
   <webots>
     <plugin type="wall_climber.cable_supervisor_plugin.CableSupervisorPlugin">

File: src/wall_climber/urdf/my_robot.urdf.xacro (robot description, xacro)
@@ -21,4 +21,17 @@
             <pen_down_position>${pen_cfg['down_position']}</pen_down_position>
         </plugin>
+        <plugin type="wall_climber.face_display_plugin.FaceDisplayPlugin">
+            <display_name>face_display</display_name>
+            <default_text>READY</default_text>
+            <text_topic>/wall_climber/face/text</text_topic>
+            <expression_topic>/wall_climber/face/expression</expression_topic>
+            <blink_period_sec>3.8</blink_period_sec>
+            <blink_duration_sec>0.14</blink_duration_sec>
+        </plugin>
+        <device reference="screen_link" type="Display">
+            <name>face_display</name>
+            <width>256</width>
+            <height>128</height>
+        </device>
     </webots>
     </robot>
