Commit message: Visual improvements: arm-exit slot, stepper-motor anchors, animated face display

File: src/wall_climber/urdf/base_body.xacro (robot description, xacro)
@@ -136,17 +136,15 @@
     <xacro:property name="service_panel_y" value="${-carriage_cfg['height'] * 0.04}"/>
     <xacro:property name="service_panel_z" value="${carriage_cfg['depth'] / 2.0 - service_panel_d / 2.0}"/>
-    <xacro:property name="arm_exit_slot_x" value="${(carriage_cfg['width'] * 0.5) - ((carriage_cfg['width'] * 0.18) * 0.5) - 0.016}"/>
+    <xacro:property name="arm_exit_slot_x" value="${carriage_cfg['width'] / 2.0 + 0.0025}"/>
     <xacro:property name="arm_exit_slot_y" value="${-carriage_cfg['pen_offset_y']}"/>
-    <xacro:property name="arm_exit_slot_w" value="${carriage_cfg['width'] * 0.26}"/>
-    <xacro:property name="arm_exit_slot_h" value="${carriage_cfg['height'] * 0.48}"/>
-    <xacro:property name="arm_exit_slot_d" value="${carriage_cfg['depth'] * 0.08}"/>
-    <xacro:property name="arm_exit_slot_z" value="${-(carriage_cfg['depth'] / 2.0) + arm_exit_slot_d / 2.0 + 0.0004}"/>
+    <xacro:property name="arm_exit_slot_w" value="0.005"/>
+    <xacro:property name="arm_exit_slot_h" value="${carriage_cfg['height'] * 0.50}"/>
+    <xacro:property name="arm_exit_slot_d" value="${carriage_cfg['depth'] * 0.48}"/>
+    <xacro:property name="arm_exit_slot_z" value="${-(carriage_cfg['depth'] / 2.0) + 0.0195}"/>
     <xacro:property name="arm_exit_bezel_t" value="0.006"/>
-    <xacro:property name="arm_exit_bezel_d" value="${carriage_cfg['depth'] * 0.07}"/>
-    <xacro:property name="arm_exit_bezel_z" value="${-(carriage_cfg['depth'] / 2.0) + arm_exit_bezel_d / 2.0 + 0.0008}"/>
-    <xacro:property name="arm_exit_rail_w" value="${arm_exit_slot_w * 0.72}"/>
+    <xacro:property name="arm_exit_bezel_x" value="${carriage_cfg['width'] / 2.0 + 0.005}"/>
+    <xacro:property name="arm_exit_rail_x" value="${carriage_cfg['width'] / 2.0 + 0.006}"/>
     <xacro:property name="arm_exit_rail_h" value="0.0036"/>
-    <xacro:property name="arm_exit_rail_d" value="${carriage_cfg['depth'] * 0.09}"/>
-    <xacro:property name="arm_exit_rail_z" value="${-(carriage_cfg['depth'] / 2.0) + arm_exit_rail_d / 2.0 + 0.0012}"/>
+    <xacro:property name="arm_exit_rail_d" value="${arm_exit_slot_d * 0.8}"/>
     <xacro:property name="vent_slit_w" value="${service_panel_w * 0.68}"/>
     <xacro:property name="vent_slit_h" value="0.0040"/>
@@ -286,7 +284,7 @@
       </visual>
       <visual>
-        <origin xyz="${arm_exit_slot_x} ${arm_exit_slot_y + arm_exit_slot_h / 2.0 + arm_exit_bezel_t / 2.0} ${arm_exit_bezel_z}" rpy="0 0 0"/>
-        <geometry>
-          <box size="${arm_exit_slot_w + 2.0 * arm_exit_bezel_t} ${arm_exit_bezel_t} ${arm_exit_bezel_d}"/>
+        <origin xyz="${arm_exit_bezel_x} ${arm_exit_slot_y + arm_exit_slot_h / 2.0 + arm_exit_bezel_t / 2.0} ${arm_exit_slot_z}" rpy="0 0 0"/>
+        <geometry>
+          <box size="0.004 ${arm_exit_bezel_t} ${arm_exit_slot_d + 2.0 * arm_exit_bezel_t}"/>
         </geometry>
         <material name="robot_arm_exit_bezel_mat">
@@ -295,7 +293,7 @@
       </visual>
       <visual>
-        <origin xyz="${arm_exit_slot_x} ${arm_exit_slot_y - arm_exit_slot_h / 2.0 - arm_exit_bezel_t / 2.0} ${arm_exit_bezel_z}" rpy="0 0 0"/>
-        <geometry>
-          <box size="${arm_exit_slot_w + 2.0 * arm_exit_bezel_t} ${arm_exit_bezel_t} ${arm_exit_bezel_d}"/>
+        <origin xyz="${arm_exit_bezel_x} ${arm_exit_slot_y - arm_exit_slot_h / 2.0 - arm_exit_bezel_t / 2.0} ${arm_exit_slot_z}" rpy="0 0 0"/>
+        <geometry>
+          <box size="0.004 ${arm_exit_bezel_t} ${arm_exit_slot_d + 2.0 * arm_exit_bezel_t}"/>
         </geometry>
         <material name="robot_arm_exit_bezel_mat">
@@ -304,7 +302,7 @@
       </visual>
       <visual>
-        <origin xyz="${arm_exit_slot_x - arm_exit_slot_w / 2.0 - arm_exit_bezel_t / 2.0} ${arm_exit_slot_y} ${arm_exit_bezel_z}" rpy="0 0 0"/>
-        <geometry>
-          <box size="${arm_exit_bezel_t} ${arm_exit_slot_h + 2.0 * arm_exit_bezel_t} ${arm_exit_bezel_d}"/>
+        <origin xyz="${arm_exit_bezel_x} ${arm_exit_slot_y} ${arm_exit_slot_z + arm_exit_slot_d / 2.0 + arm_exit_bezel_t / 2.0}" rpy="0 0 0"/>
+        <geometry>
+          <box size="0.004 ${arm_exit_slot_h} ${arm_exit_bezel_t}"/>
         </geometry>
         <material name="robot_arm_exit_bezel_mat">
@@ -313,7 +311,7 @@
       </visual>
       <visual>
-        <origin xyz="${arm_exit_slot_x + arm_exit_slot_w / 2.0 + arm_exit_bezel_t / 2.0} ${arm_exit_slot_y} ${arm_exit_bezel_z}" rpy="0 0 0"/>
-        <geometry>
-          <box size="${arm_exit_bezel_t} ${arm_exit_slot_h + 2.0 * arm_exit_bezel_t} ${arm_exit_bezel_d}"/>
+        <origin xyz="${arm_exit_bezel_x} ${arm_exit_slot_y} ${arm_exit_slot_z - arm_exit_slot_d / 2.0 - arm_exit_bezel_t / 2.0}" rpy="0 0 0"/>
+        <geometry>
+          <box size="0.004 ${arm_exit_slot_h} ${arm_exit_bezel_t}"/>
         </geometry>
         <material name="robot_arm_exit_bezel_mat">
@@ -322,7 +320,7 @@
       </visual>
       <visual>
-        <origin xyz="${arm_exit_slot_x} ${arm_exit_slot_y + arm_exit_slot_h * 0.22} ${arm_exit_rail_z}" rpy="0 0 0"/>
-        <geometry>
-          <box size="${arm_exit_rail_w} ${arm_exit_rail_h} ${arm_exit_rail_d}"/>
+        <origin xyz="${arm_exit_rail_x} ${arm_exit_slot_y + arm_exit_slot_h * 0.24} ${arm_exit_slot_z}" rpy="0 0 0"/>
+        <geometry>
+          <box size="0.003 ${arm_exit_rail_h} ${arm_exit_rail_d}"/>
         </geometry>
         <material name="robot_arm_exit_rail_mat">
@@ -331,7 +329,7 @@
       </visual>
       <visual>
-        <origin xyz="${arm_exit_slot_x} ${arm_exit_slot_y - arm_exit_slot_h * 0.22} ${arm_exit_rail_z}" rpy="0 0 0"/>
-        <geometry>
-          <box size="${arm_exit_rail_w} ${arm_exit_rail_h} ${arm_exit_rail_d}"/>
+        <origin xyz="${arm_exit_rail_x} ${arm_exit_slot_y - arm_exit_slot_h * 0.24} ${arm_exit_slot_z}" rpy="0 0 0"/>
+        <geometry>
+          <box size="0.003 ${arm_exit_rail_h} ${arm_exit_rail_d}"/>
         </geometry>
         <material name="robot_arm_exit_rail_mat">

File: src/wall_climber/urdf/cable_supervisor.urdf.xacro (robot description, xacro)
@@ -36,5 +36,5 @@
         <origin xyz="${0.018 * x_sign} 0.010 ${0.018 * z_sign}" rpy="0 0 0"/>
         <geometry>
-          <box size="0.050 0.007 0.050"/>
+          <box size="0.040 0.006 0.040"/>
         </geometry>
         <material name="${name}_mounting_plate_mat">
@@ -43,16 +43,16 @@
       </visual>
       <visual>
-        <origin xyz="${0.018 * x_sign} 0.025 ${0.018 * z_sign}" rpy="0 0 0"/>
-        <geometry>
-          <box size="0.038 0.026 0.038"/>
+        <origin xyz="${0.018 * x_sign} 0.028 ${0.018 * z_sign}" rpy="0 0 0"/>
+        <geometry>
+          <box size="0.034 0.030 0.034"/>
         </geometry>
         <material name="${name}_motor_housing_mat">
-          <color rgba="0.23 0.26 0.31 1.0"/>
-        </material>
-      </visual>
-      <visual>
-        <origin xyz="${0.018 * x_sign} 0.040 ${0.018 * z_sign}" rpy="0 0 0"/>
-        <geometry>
-          <box size="0.041 0.0045 0.041"/>
+          <color rgba="0.08 0.09 0.11 1.0"/>
+        </material>
+      </visual>
+      <visual>
+        <origin xyz="${0.018 * x_sign} 0.028 ${0.018 * z_sign}" rpy="0 0 0"/>
+        <geometry>
+          <box size="0.035 0.004 0.035"/>
         </geometry>
         <material name="${name}_accent_band_mat">
@@ -61,36 +61,36 @@
       </visual>
       <visual>
-        <origin xyz="${0.041 * x_sign} 0.027 ${0.018 * z_sign}" rpy="0 0 0"/>
-        <geometry>
-          <box size="0.011 0.018 0.016"/>
+        <origin xyz="${0.018 * x_sign} 0.044 ${0.018 * z_sign}" rpy="0 0 0"/>
+        <geometry>
+          <box size="0.012 0.004 0.012"/>
         </geometry>
         <material name="${name}_connector_cap_mat">
-          <color rgba="0.08 0.09 0.11 1.0"/>
-        </material>
-      </visual>
-      <visual>
-        <origin xyz="${0.018 * x_sign - 0.013} 0.044 ${0.018 * z_sign - 0.013}" rpy="1.57079632679 0 0"/>
-        <geometry><cylinder radius="0.0028" length="0.004"/></geometry>
-        <material name="${name}_bolt_mat"><color rgba="0.70 0.74 0.80 1.0"/></material>
-      </visual>
-      <visual>
-        <origin xyz="${0.018 * x_sign + 0.013} 0.044 ${0.018 * z_sign - 0.013}" rpy="1.57079632679 0 0"/>
-        <geometry><cylinder radius="0.0028" length="0.004"/></geometry>
-        <material name="${name}_bolt_mat"><color rgba="0.70 0.74 0.80 1.0"/></material>
-      </visual>
-      <visual>
-        <origin xyz="${0.018 * x_sign - 0.013} 0.044 ${0.018 * z_sign + 0.013}" rpy="1.57079632679 0 0"/>
-        <geometry><cylinder radius="0.0028" length="0.004"/></geometry>
-        <material name="${name}_bolt_mat"><color rgba="0.70 0.74 0.80 1.0"/></material>
-      </visual>
-      <visual>
-        <origin xyz="${0.018 * x_sign + 0.013} 0.044 ${0.018 * z_sign + 0.013}" rpy="1.57079632679 0 0"/>
-        <geometry><cylinder radius="0.0028" length="0.004"/></geometry>
-        <material name="${name}_bolt_mat"><color rgba="0.70 0.74 0.80 1.0"/></material>
-      </visual>
-      <visual>
-        <origin xyz="0 0.043 0" rpy="1.57079632679 0 0"/>
-        <geometry>
-          <cylinder radius="0.0048" length="0.014"/>
+          <color rgba="0.12 0.14 0.17 1.0"/>
+        </material>
+      </visual>
+      <visual>
+        <origin xyz="${0.018 * x_sign - 0.014} 0.014 ${0.018 * z_sign - 0.014}" rpy="1.57079632679 0 0"/>
+        <geometry><cylinder radius="0.0025" length="0.003"/></geometry>
+        <material name="${name}_bolt_mat"><color rgba="0.70 0.74 0.80 1.0"/></material>
+      </visual>
+      <visual>
+        <origin xyz="${0.018 * x_sign + 0.014} 0.014 ${0.018 * z_sign - 0.014}" rpy="1.57079632679 0 0"/>
+        <geometry><cylinder radius="0.0025" length="0.003"/></geometry>
+        <material name="${name}_bolt_mat"><color rgba="0.70 0.74 0.80 1.0"/></material>
+      </visual>
+      <visual>
+        <origin xyz="${0.018 * x_sign - 0.014} 0.014 ${0.018 * z_sign + 0.014}" rpy="1.57079632679 0 0"/>
+        <geometry><cylinder radius="0.0025" length="0.003"/></geometry>
+        <material name="${name}_bolt_mat"><color rgba="0.70 0.74 0.80 1.0"/></material>
+      </visual>
+      <visual>
+        <origin xyz="${0.018 * x_sign + 0.014} 0.014 ${0.018 * z_sign + 0.014}" rpy="1.57079632679 0 0"/>
+        <geometry><cylinder radius="0.0025" length="0.003"/></geometry>
+        <material name="${name}_bolt_mat"><color rgba="0.70 0.74 0.80 1.0"/></material>
+      </visual>
+      <visual>
+        <origin xyz="0 0.008 0" rpy="1.57079632679 0 0"/>
+        <geometry>
+          <cylinder radius="0.004" length="0.012"/>
         </geometry>
         <material name="${name}_output_shaft_mat">
@@ -99,7 +99,7 @@
       </visual>
       <visual>
-        <origin xyz="0 0.052 0" rpy="1.57079632679 0 0"/>
-        <geometry>
-          <cylinder radius="0.0135" length="0.011"/>
+        <origin xyz="0 0.002 0" rpy="1.57079632679 0 0"/>
+        <geometry>
+          <cylinder radius="0.014" length="0.008"/>
         </geometry>
         <material name="${name}_pulley_mat">
@@ -108,7 +108,7 @@
       </visual>
       <visual>
-        <origin xyz="0 0.052 0" rpy="1.57079632679 0 0"/>
-        <geometry>
-          <cylinder radius="0.0142" length="0.0022"/>
+        <origin xyz="0 0.002 0" rpy="1.57079632679 0 0"/>
+        <geometry>
+          <cylinder radius="0.015" length="0.002"/>
         </geometry>
         <material name="${name}_pulley_groove_mat">
@@ -117,7 +117,7 @@
       </visual>
       <visual>
-        <origin xyz="0 0.059 0" rpy="1.57079632679 0 0"/>
-        <geometry>
-          <cylinder radius="0.0065" length="0.006"/>
+        <origin xyz="0 -0.004 0" rpy="1.57079632679 0 0"/>
+        <geometry>
+          <cylinder radius="0.006" length="0.004"/>
         </geometry>
         <material name="${name}_pulley_hub_mat">
@@ -132,8 +132,8 @@
   </xacro:macro>
   <link name="base_link"/>
-  <xacro:board_anchor_visual name="left_board_anchor" world_x="${left_anchor_world_x}" world_z="${left_anchor_world_z}" x_sign="1" z_sign="-1"/>
-  <xacro:board_anchor_visual name="right_board_anchor" world_x="${right_anchor_world_x}" world_z="${right_anchor_world_z}" x_sign="-1" z_sign="-1"/>
-  <xacro:board_anchor_visual name="bottom_left_board_anchor" world_x="${bottom_left_anchor_world_x}" world_z="${bottom_left_anchor_world_z}" x_sign="1" z_sign="1"/>
-  <xacro:board_anchor_visual name="bottom_right_board_anchor" world_x="${bottom_right_anchor_world_x}" world_z="${bottom_right_anchor_world_z}" x_sign="-1" z_sign="1"/>
+  <xacro:board_anchor_visual name="left_board_anchor" world_x="${left_anchor_world_x}" world_z="${left_anchor_world_z}" x_sign="-1" z_sign="-1"/>
+  <xacro:board_anchor_visual name="right_board_anchor" world_x="${right_anchor_world_x}" world_z="${right_anchor_world_z}" x_sign="1" z_sign="-1"/>
+  <xacro:board_anchor_visual name="bottom_left_board_anchor" world_x="${bottom_left_anchor_world_x}" world_z="${bottom_left_anchor_world_z}" x_sign="-1" z_sign="1"/>
+  <xacro:board_anchor_visual name="bottom_right_board_anchor" world_x="${bottom_right_anchor_world_x}" world_z="${bottom_right_anchor_world_z}" x_sign="1" z_sign="1"/>
   <webots>
     <plugin type="wall_climber.cable_supervisor_plugin.CableSupervisorPlugin">

File: src/wall_climber/urdf/robot_face_screen.xacro (robot description, xacro)
@@ -1,4 +1,4 @@
 <?xml version="1.0"?>
-<robot xmlns:xacro="http://www.ros.org/wiki/xacro">
+<robot xmlns:xacro="http://www.ros.org/wiki/xacro" xmlns:webots="http://www.cyberbotics.com">
   <xacro:macro name="rounded_panel" params="x y z width height depth radius mat_name rgba">
     <visual>
@@ -116,16 +116,22 @@
     </joint>
     <link name="screen_link">
-      <xacro:rounded_panel
-        x="0" y="0" z="0"
-        width="${bezel_width}" height="${bezel_height}" depth="${bezel_depth}" radius="${bezel_radius}"
-        mat_name="screen_bezel_mat" rgba="0.02 0.03 0.04 1.0"/>
-      <xacro:rounded_panel
-        x="0" y="0" z="${bezel_depth / 2.0 + screen_depth / 2.0 - 0.0004}"
-        width="${screen_width}" height="${screen_height}" depth="${screen_depth}" radius="${screen_radius}"
-        mat_name="screen_glass_mat" rgba="0.03 0.10 0.14 1.0"/>
-      <xacro:rounded_panel
-        x="0" y="0" z="${bezel_depth / 2.0 + screen_depth + 0.0002}"
-        width="${screen_width * 0.96}" height="${screen_height * 0.96}" depth="0.0008" radius="${screen_radius * 0.92}"
-        mat_name="screen_emit_mat" rgba="0.05 0.84 0.92 1.0"/>
+      <visual>
+        <origin xyz="0 0 0" rpy="0 0 0"/>
+        <geometry>
+          <box size="${bezel_width} ${bezel_height} ${bezel_depth}"/>
+        </geometry>
+        <material name="screen_bezel_mat">
+          <color rgba="0.02 0.03 0.04 1.0"/>
+        </material>
+      </visual>
+      <visual>
+        <origin xyz="0 0 ${bezel_depth / 2.0 + 0.0001}" rpy="0 0 0"/>
+        <geometry>
+          <box size="${screen_width} ${screen_height} 0.001"/>
+        </geometry>
+        <material name="screen_glass_mat">
+          <color rgba="0.01 0.01 0.01 1.0"/>
+        </material>
+      </visual>
       <collision>
         <geometry>
@@ -137,4 +143,5 @@
         <inertia ixx="0.00001" ixy="0" ixz="0" iyy="0.00001" iyz="0" izz="0.00001"/>
       </inertial>
+      <webots:device reference="face_display" type="Display"/>
     </link>
   </xacro:macro>
