Commit message: Add four-cable kinematics draft

File: src/wall_climber/urdf/cable_supervisor.urdf.xacro (robot description, xacro)
@@ -13,13 +13,17 @@
   <xacro:property name="safe_y_max" value="${board_cfg['height'] - board_cfg['margin_bottom'] - workspace_cfg['safety_margin_bottom']}"/>
   <xacro:property name="chassis_root_local_z" value="${carriage_cfg['root_to_chassis_z']}"/>
-  <xacro:property name="cable_mount_left_local_y" value="${-carriage_cfg['attachment_left_y']}"/>
-  <xacro:property name="cable_mount_right_local_y" value="${-carriage_cfg['attachment_right_y']}"/>
+  <xacro:property name="cable_mount_left_local_y" value="${-carriage_cfg['attachment_top_left_y']}"/>
+  <xacro:property name="cable_mount_right_local_y" value="${-carriage_cfg['attachment_top_right_y']}"/>
   <xacro:property name="cable_mount_local_z" value="${chassis_root_local_z - (carriage_cfg['depth'] / 2.0) + 0.002}"/>
   <xacro:property name="board_left_world_x" value="${board_cfg['center_x'] - (board_cfg['width'] / 2.0)}"/>
   <xacro:property name="board_top_world_z" value="${board_cfg['center_z'] + (board_cfg['height'] / 2.0)}"/>
-  <xacro:property name="left_anchor_world_x" value="${board_left_world_x + anchor_cfg['left_x']}"/>
-  <xacro:property name="left_anchor_world_z" value="${board_top_world_z - anchor_cfg['left_y']}"/>
-  <xacro:property name="right_anchor_world_x" value="${board_left_world_x + anchor_cfg['right_x']}"/>
-  <xacro:property name="right_anchor_world_z" value="${board_top_world_z - anchor_cfg['right_y']}"/>
+  <xacro:property name="left_anchor_world_x" value="${board_left_world_x + anchor_cfg['top_left_x']}"/>
+  <xacro:property name="left_anchor_world_z" value="${board_top_world_z - anchor_cfg['top_left_y']}"/>
+  <xacro:property name="right_anchor_world_x" value="${board_left_world_x + anchor_cfg['top_right_x']}"/>
+  <xacro:property name="right_anchor_world_z" value="${board_top_world_z - anchor_cfg['top_right_y']}"/>
+  <xacro:property name="bottom_left_anchor_world_x" value="${board_left_world_x + anchor_cfg['bottom_left_x']}"/>
+  <xacro:property name="bottom_left_anchor_world_z" value="${board_top_world_z - anchor_cfg['bottom_left_y']}"/>
+  <xacro:property name="bottom_right_anchor_world_x" value="${board_left_world_x + anchor_cfg['bottom_right_x']}"/>
+  <xacro:property name="bottom_right_anchor_world_z" value="${board_top_world_z - anchor_cfg['bottom_right_y']}"/>
   <xacro:macro name="board_anchor_visual" params="name world_x world_z x_sign">
     <joint name="${name}_joint" type="fixed">
@@ -74,4 +78,6 @@
   <xacro:board_anchor_visual name="left_board_anchor" world_x="${left_anchor_world_x}" world_z="${left_anchor_world_z}" x_sign="1"/>
   <xacro:board_anchor_visual name="right_board_anchor" world_x="${right_anchor_world_x}" world_z="${right_anchor_world_z}" x_sign="-1"/>
+  <xacro:board_anchor_visual name="bottom_left_board_anchor" world_x="${bottom_left_anchor_world_x}" world_z="${bottom_left_anchor_world_z}" x_sign="1"/>
+  <xacro:board_anchor_visual name="bottom_right_board_anchor" world_x="${bottom_right_anchor_world_x}" world_z="${bottom_right_anchor_world_z}" x_sign="-1"/>
   <webots>
     <plugin type="wall_climber.cable_supervisor_plugin.CableSupervisorPlugin">
@@ -93,8 +99,24 @@
       <safe_y_max>${safe_y_max}</safe_y_max>
       <corner_keepout_radius>${workspace_cfg['corner_keepout_radius']}</corner_keepout_radius>
+      <anchor_top_left_x>${anchor_cfg['top_left_x']}</anchor_top_left_x>
+      <anchor_top_left_y>${anchor_cfg['top_left_y']}</anchor_top_left_y>
+      <anchor_top_right_x>${anchor_cfg['top_right_x']}</anchor_top_right_x>
+      <anchor_top_right_y>${anchor_cfg['top_right_y']}</anchor_top_right_y>
+      <anchor_bottom_left_x>${anchor_cfg['bottom_left_x']}</anchor_bottom_left_x>
+      <anchor_bottom_left_y>${anchor_cfg['bottom_left_y']}</anchor_bottom_left_y>
+      <anchor_bottom_right_x>${anchor_cfg['bottom_right_x']}</anchor_bottom_right_x>
+      <anchor_bottom_right_y>${anchor_cfg['bottom_right_y']}</anchor_bottom_right_y>
       <anchor_left_x>${anchor_cfg['left_x']}</anchor_left_x>
       <anchor_left_y>${anchor_cfg['left_y']}</anchor_left_y>
       <anchor_right_x>${anchor_cfg['right_x']}</anchor_right_x>
       <anchor_right_y>${anchor_cfg['right_y']}</anchor_right_y>
+      <carriage_attachment_top_left_x>${carriage_cfg['attachment_top_left_x']}</carriage_attachment_top_left_x>
+      <carriage_attachment_top_left_y>${carriage_cfg['attachment_top_left_y']}</carriage_attachment_top_left_y>
+      <carriage_attachment_top_right_x>${carriage_cfg['attachment_top_right_x']}</carriage_attachment_top_right_x>
+      <carriage_attachment_top_right_y>${carriage_cfg['attachment_top_right_y']}</carriage_attachment_top_right_y>
+      <carriage_attachment_bottom_left_x>${carriage_cfg['attachment_bottom_left_x']}</carriage_attachment_bottom_left_x>
+      <carriage_attachment_bottom_left_y>${carriage_cfg['attachment_bottom_left_y']}</carriage_attachment_bottom_left_y>
+      <carriage_attachment_bottom_right_x>${carriage_cfg['attachment_bottom_right_x']}</carriage_attachment_bottom_right_x>
+      <carriage_attachment_bottom_right_y>${carriage_cfg['attachment_bottom_right_y']}</carriage_attachment_bottom_right_y>
       <carriage_attachment_left_x>${carriage_cfg['attachment_left_x']}</carriage_attachment_left_x>
       <carriage_attachment_left_y>${carriage_cfg['attachment_left_y']}</carriage_attachment_left_y>
@@ -103,7 +125,7 @@
       <carriage_width>${carriage_cfg['width']}</carriage_width>
       <carriage_height>${carriage_cfg['height']}</carriage_height>
-      <cable_mount_left_local_x>${carriage_cfg['attachment_left_x']}</cable_mount_left_local_x>
+      <cable_mount_left_local_x>${carriage_cfg['attachment_top_left_x']}</cable_mount_left_local_x>
       <cable_mount_left_local_y>${cable_mount_left_local_y}</cable_mount_left_local_y>
-      <cable_mount_right_local_x>${carriage_cfg['attachment_right_x']}</cable_mount_right_local_x>
+      <cable_mount_right_local_x>${carriage_cfg['attachment_top_right_x']}</cable_mount_right_local_x>
       <cable_mount_right_local_y>${cable_mount_right_local_y}</cable_mount_right_local_y>
       <cable_mount_local_z>${cable_mount_local_z}</cable_mount_local_z>

Commit message: Fix: Corner motor visibility and screen display mapping

File: src/wall_climber/urdf/cable_supervisor.urdf.xacro (robot description, xacro)
@@ -30,9 +30,11 @@
       <parent link="base_link"/>
       <child link="${name}"/>
-      <origin xyz="${world_x} ${board_cfg['surface_y']} ${world_z}" rpy="0 0 0"/>
+      <!-- Move anchor origin forward (smaller Y) to be in front of the frame -->
+      <origin xyz="${world_x} ${board_cfg['surface_y'] - 0.035} ${world_z}" rpy="0 0 0"/>
     </joint>
     <link name="${name}">
       <visual>
-        <origin xyz="${0.018 * x_sign} 0.010 ${0.018 * z_sign}" rpy="0 0 0"/>
+        <!-- Negative Y offsets move elements away from the wall -->
+        <origin xyz="${0.018 * x_sign} -0.005 ${0.018 * z_sign}" rpy="0 0 0"/>
         <geometry>
           <box size="0.040 0.006 0.040"/>
@@ -43,5 +45,5 @@
       </visual>
       <visual>
-        <origin xyz="${0.018 * x_sign} 0.028 ${0.018 * z_sign}" rpy="0 0 0"/>
+        <origin xyz="${0.018 * x_sign} -0.023 ${0.018 * z_sign}" rpy="0 0 0"/>
         <geometry>
           <box size="0.034 0.030 0.034"/>
@@ -52,5 +54,5 @@
       </visual>
       <visual>
-        <origin xyz="${0.018 * x_sign} 0.028 ${0.018 * z_sign}" rpy="0 0 0"/>
+        <origin xyz="${0.018 * x_sign} -0.023 ${0.018 * z_sign}" rpy="0 0 0"/>
         <geometry>
           <box size="0.035 0.004 0.035"/>
@@ -61,5 +63,5 @@
       </visual>
       <visual>
-        <origin xyz="${0.018 * x_sign} 0.044 ${0.018 * z_sign}" rpy="0 0 0"/>
+        <origin xyz="${0.018 * x_sign} -0.039 ${0.018 * z_sign}" rpy="0 0 0"/>
         <geometry>
           <box size="0.012 0.004 0.012"/>
@@ -70,25 +72,25 @@
       </visual>
       <visual>
-        <origin xyz="${0.018 * x_sign - 0.014} 0.014 ${0.018 * z_sign - 0.014}" rpy="1.57079632679 0 0"/>
-        <geometry><cylinder radius="0.0025" length="0.003"/></geometry>
-        <material name="${name}_bolt_mat"><color rgba="0.70 0.74 0.80 1.0"/></material>
-      </visual>
-      <visual>
-        <origin xyz="${0.018 * x_sign + 0.014} 0.014 ${0.018 * z_sign - 0.014}" rpy="1.57079632679 0 0"/>
-        <geometry><cylinder radius="0.0025" length="0.003"/></geometry>
-        <material name="${name}_bolt_mat"><color rgba="0.70 0.74 0.80 1.0"/></material>
-      </visual>
-      <visual>
-        <origin xyz="${0.018 * x_sign - 0.014} 0.014 ${0.018 * z_sign + 0.014}" rpy="1.57079632679 0 0"/>
-        <geometry><cylinder radius="0.0025" length="0.003"/></geometry>
-        <material name="${name}_bolt_mat"><color rgba="0.70 0.74 0.80 1.0"/></material>
-      </visual>
-      <visual>
-        <origin xyz="${0.018 * x_sign + 0.014} 0.014 ${0.018 * z_sign + 0.014}" rpy="1.57079632679 0 0"/>
-        <geometry><cylinder radius="0.0025" length="0.003"/></geometry>
-        <material name="${name}_bolt_mat"><color rgba="0.70 0.74 0.80 1.0"/></material>
-      </visual>
-      <visual>
-        <origin xyz="0 0.008 0" rpy="1.57079632679 0 0"/>
+        <origin xyz="${0.018 * x_sign - 0.014} -0.009 ${0.018 * z_sign - 0.014}" rpy="1.57079632679 0 0"/>
+        <geometry><cylinder radius="0.0025" length="0.003"/></geometry>
+        <material name="${name}_bolt_mat"><color rgba="0.70 0.74 0.80 1.0"/></material>
+      </visual>
+      <visual>
+        <origin xyz="${0.018 * x_sign + 0.014} -0.009 ${0.018 * z_sign - 0.014}" rpy="1.57079632679 0 0"/>
+        <geometry><cylinder radius="0.0025" length="0.003"/></geometry>
+        <material name="${name}_bolt_mat"><color rgba="0.70 0.74 0.80 1.0"/></material>
+      </visual>
+      <visual>
+        <origin xyz="${0.018 * x_sign - 0.014} -0.009 ${0.018 * z_sign + 0.014}" rpy="1.57079632679 0 0"/>
+        <geometry><cylinder radius="0.0025" length="0.003"/></geometry>
+        <material name="${name}_bolt_mat"><color rgba="0.70 0.74 0.80 1.0"/></material>
+      </visual>
+      <visual>
+        <origin xyz="${0.018 * x_sign + 0.014} -0.009 ${0.018 * z_sign + 0.014}" rpy="1.57079632679 0 0"/>
+        <geometry><cylinder radius="0.0025" length="0.003"/></geometry>
+        <material name="${name}_bolt_mat"><color rgba="0.70 0.74 0.80 1.0"/></material>
+      </visual>
+      <visual>
+        <origin xyz="0 -0.003 0" rpy="1.57079632679 0 0"/>
         <geometry>
           <cylinder radius="0.004" length="0.012"/>
@@ -99,5 +101,5 @@
       </visual>
       <visual>
-        <origin xyz="0 0.002 0" rpy="1.57079632679 0 0"/>
+        <origin xyz="0 0.003 0" rpy="1.57079632679 0 0"/>
         <geometry>
           <cylinder radius="0.014" length="0.008"/>
@@ -108,5 +110,5 @@
       </visual>
       <visual>
-        <origin xyz="0 0.002 0" rpy="1.57079632679 0 0"/>
+        <origin xyz="0 0.003 0" rpy="1.57079632679 0 0"/>
         <geometry>
           <cylinder radius="0.015" length="0.002"/>
@@ -117,5 +119,5 @@
       </visual>
       <visual>
-        <origin xyz="0 -0.004 0" rpy="1.57079632679 0 0"/>
+        <origin xyz="0 0.009 0" rpy="1.57079632679 0 0"/>
         <geometry>
           <cylinder radius="0.006" length="0.004"/>
@@ -132,8 +134,10 @@
   </xacro:macro>
   <link name="base_link"/>
-  <xacro:board_anchor_visual name="left_board_anchor" world_x="${left_anchor_world_x}" world_z="${left_anchor_world_z}" x_sign="-1" z_sign="-1"/>
-  <xacro:board_anchor_visual name="right_board_anchor" world_x="${right_anchor_world_x}" world_z="${right_anchor_world_z}" x_sign="1" z_sign="-1"/>
-  <xacro:board_anchor_visual name="bottom_left_board_anchor" world_x="${bottom_left_anchor_world_x}" world_z="${bottom_left_anchor_world_z}" x_sign="-1" z_sign="1"/>
-  <xacro:board_anchor_visual name="bottom_right_board_anchor" world_x="${bottom_right_anchor_world_x}" world_z="${bottom_right_anchor_world_z}" x_sign="1" z_sign="1"/>
+  <!-- x_sign=1 moves inward for left anchors, x_sign=-1 moves inward for right anchors -->
+  <!-- z_sign=-1 moves inward (down) for top anchors, z_sign=1 moves inward (up) for bottom anchors -->
+  <xacro:board_anchor_visual name="left_board_anchor" world_x="${left_anchor_world_x}" world_z="${left_anchor_world_z}" x_sign="1" z_sign="-1"/>
+  <xacro:board_anchor_visual name="right_board_anchor" world_x="${right_anchor_world_x}" world_z="${right_anchor_world_z}" x_sign="-1" z_sign="-1"/>
+  <xacro:board_anchor_visual name="bottom_left_board_anchor" world_x="${bottom_left_anchor_world_x}" world_z="${bottom_left_anchor_world_z}" x_sign="1" z_sign="1"/>
+  <xacro:board_anchor_visual name="bottom_right_board_anchor" world_x="${bottom_right_anchor_world_x}" world_z="${bottom_right_anchor_world_z}" x_sign="-1" z_sign="1"/>
   <webots>
     <plugin type="wall_climber.cable_supervisor_plugin.CableSupervisorPlugin">

File: src/wall_climber/urdf/robot_face_screen.xacro (robot description, xacro)
@@ -130,5 +130,6 @@
           <box size="${screen_width} ${screen_height} 0.001"/>
         </geometry>
-        <material name="screen_glass_mat">
+        <!-- The material name MUST match the device name for Webots to map the Display -->
+        <material name="face_display">
           <color rgba="0.01 0.01 0.01 1.0"/>
         </material>
